Commit message: Edited single_motor_test urdf

File: src/meldog_hardware/pi3hat_hardware_interface/test/test_single_motor.urdf.xacro (robot description, xacro)
@@ -7,12 +7,12 @@
         <inertia ixx="0.001" ixy="0" ixz="0" iyy="0.001" iyz="0" izz="0.001"/>
     </inertial>
-    <visual name="Cube">
+    <visual>
         <origin xyz="0 0 0" rpy="0 0 0"/>
         <geometry>
-        <box size="0.24 0.14 0.22"/>
+        <box size="0.25 0.25 0.25"/>
         </geometry>
     </visual>
   </link>
-  <link name="link_1">
+  <link name="rotor">
     <inertial>
         <origin xyz="0 0 0" rpy="0 0 0"/>
@@ -20,15 +20,15 @@
         <inertia ixx="0.001" ixy="0" ixz="0" iyy="0.001" iyz="0" izz="0.001"/>
     </inertial>
-    <visual name="Cube">
+    <visual>
         <origin xyz="0 0 0" rpy="0 0 0"/>
         <geometry>
-        <box size="0.24 0.14 0.22"/>
+          <cylinder radius="0.125" length="0.05"/>
         </geometry>
     </visual>
   </link>
   <joint name="joint_1" type="revolute">
-        <origin xyz="0 -0.1 0" rpy="1.5708 1.5708 0"/>
+        <origin xyz="0.15 0 0" rpy="0 0 0"/>
         <parent link="base_link"/>
-        <child link="link_1"/>
+        <child link="rotor"/>
         <axis xyz="0 0 1.0"/>
         <limit lower="-1.39626" upper="-0.5236" effort="35.0" velocity="26.0"/>
@@ -45,4 +45,22 @@
         <parent link="base_link"/>
         <child link="imu"/>
+  </joint>
+  <link name="indicator">
+    <inertial>
+        <origin xyz="0 0 0" rpy="0 0 0"/>
+        <mass value="0.001"/>
+        <inertia ixx="0.001" ixy="0" ixz="0" iyy="0.001" iyz="0" izz="0.001"/>
+    </inertial>
+    <visual>
+      <geometry>
+        <origin xyz="0 0 0" rpy="0 0 0"/>
+        <box size="0.01 0.01 0.1"/>
+      </geometry>
+    </visual>
+  </link>
+  <joint name="rotor_indicator_joint" type="fixed">
+        <origin xyz="0.025 0 0.05" rpy="1.5708 0 1.5708"/>
+        <parent link="rotor"/>
+        <child link="indicator"/>
   </joint>
   <ros2_control name="pi3hat_hardware_interface" type="system">
