Commit message: Changed launch file

File: src/meldog_hardware/pi3hat_hardware_interface/test/urdf/test_single_motor.urdf.xacro (robot description, xacro)
@@ -28,9 +28,9 @@
   </link>
   <joint name="joint_1" type="revolute">
-        <origin xyz="0.15 0 0" rpy="0 0 0"/>
-        <parent link="base_link"/>
-        <child link="rotor"/>
-        <axis xyz="0 0 1.0"/>
-        <limit lower="-1.39626" upper="-0.5236" effort="35.0" velocity="26.0"/>
+    <origin xyz="0.0 0.0 0.0" rpy="0.0 0.0 0.0"/>
+    <parent link="base_link"/>
+    <child link="rotor"/>
+    <axis xyz="1.0 0.0 0.0"/>
+    <limit lower="-5.0" upper="5.0" effort="10.0" velocity="10.0"/>
   </joint>
   <link name="imu">

Commit message: New changes for testing on pi3hat

File: src/meldog_hardware/pi3hat_hardware_interface/test/urdf/test_single_motor.urdf.xacro (robot description, xacro)
@@ -1,67 +1,50 @@
 <?xml version="1.0"?>
 <robot xmlns:xacro="http://www.ros.org/wiki/xacro" name="test_single_motor">
-  <link name="base_link">
-    <inertial>
-        <origin xyz="0 0 0" rpy="0 0 0"/>
-        <mass value="3.0"/>
-        <inertia ixx="0.001" ixy="0" ixz="0" iyy="0.001" iyz="0" izz="0.001"/>
-    </inertial>
-    <visual>
-        <origin xyz="0 0 0" rpy="0 0 0"/>
-        <geometry>
-        <box size="0.25 0.25 0.25"/>
-        </geometry>
-    </visual>
-  </link>
-  <link name="rotor">
-    <inertial>
-        <origin xyz="0 0 0" rpy="0 0 0"/>
-        <mass value="3.0"/>
-        <inertia ixx="0.001" ixy="0" ixz="0" iyy="0.001" iyz="0" izz="0.001"/>
-    </inertial>
-    <visual>
-        <origin xyz="0 0 0" rpy="0 0 0"/>
-        <geometry>
-          <cylinder radius="0.125" length="0.05"/>
-        </geometry>
-    </visual>
-  </link>
-  <joint name="joint_1" type="revolute">
-    <origin xyz="0.0 0.0 0.0" rpy="0.0 0.0 0.0"/>
-    <parent link="base_link"/>
-    <child link="rotor"/>
-    <axis xyz="1.0 0.0 0.0"/>
-    <limit lower="-5.0" upper="5.0" effort="10.0" velocity="10.0"/>
-  </joint>
-  <link name="imu">
-    <inertial>
-        <origin xyz="0 0 0" rpy="0 0 0"/>
-        <mass value="0.001"/>
-        <inertia ixx="0.001" ixy="0" ixz="0" iyy="0.001" iyz="0" izz="0.001"/>
-    </inertial>
-  </link>
-  <joint name="imu" type="fixed">
-        <origin xyz="0 0 0" rpy="1.5708 0 1.5708"/>
-        <parent link="base_link"/>
-        <child link="imu"/>
-  </joint>
-  <link name="indicator">
-    <inertial>
-        <origin xyz="0 0 0" rpy="0 0 0"/>
-        <mass value="0.001"/>
-        <inertia ixx="0.001" ixy="0" ixz="0" iyy="0.001" iyz="0" izz="0.001"/>
-    </inertial>
-    <visual>
-      <geometry>
-        <origin xyz="0 0 0" rpy="0 0 0"/>
-        <box size="0.01 0.01 0.1"/>
-      </geometry>
-    </visual>
-  </link>
-  <joint name="rotor_indicator_joint" type="fixed">
-        <origin xyz="0.025 0 0.05" rpy="1.5708 0 1.5708"/>
+  <link name="box">
+        <visual>
+            <origin xyz="0.0 0.0 0.0" rpy="0.0 0.0 0.0"/>
+            <geometry>
+                <box size="0.5 0.5 0.5"/>
+            </geometry>
+            <material name="red">
+                <color rgba="1.0 0.0 0.0 1.0"/>
+            </material>
+        </visual>
+    </link>
+    <link name="rotor">
+        <visual>
+            <origin xyz="0.0 0.0 0.0" rpy="0.0 0.0 0.0"/>
+            <geometry>
+                <cylinder radius="0.2" length="0.1"/>
+            </geometry>
+            <material name="red">
+                <color rgba="0.0 0.0 1.0 1.0"/>
+            </material>
+        </visual>
+    </link>
+    <link name="indicator">
+        <visual>
+            <origin xyz="0.0 0.0 0.0" rpy="0.0 0.0 0.0"/>
+            <geometry>
+                <box size="0.01 0.3 0.01"/>
+            </geometry>
+            <material name="">
+                <color rgba="0.0 1.0 0.0 1.0"/>
+                <texture filename=""/>
+            </material>
+        </visual>
+    </link>
+    <joint name="joint_1" type="revolute">
+        <origin xyz="0.0 0.3 0.0" rpy="-1.5707 0.0 0.0"/>
+        <parent link="box"/>
+        <child link="rotor"/>
+        <axis xyz="0.0 0.0 -1.0"/>
+        <limit lower="-10.0" upper="10.0" effort="10.0" velocity="100.0"/>
+    </joint>
+    <joint name="joint_2" type="fixed">
+        <origin xyz="0.0 -0.25 0.055" rpy="0.0 0.0 0.0"/>
         <parent link="rotor"/>
         <child link="indicator"/>
-  </joint>
+    </joint>
   <ros2_control name="pi3hat_hardware_interface" type="system">
         <hardware>
@@ -94,5 +77,5 @@
         <actuator name="actuator_1" role="actuator1"/>
         <joint name="joint_1" role="joint1">
-            <mechanical_reduction>2.0</mechanical_reduction>
+            <mechanical_reduction>16.0</mechanical_reduction>
             <offset>0.0</offset>
         </joint>
