Commit message: Added inertial properties and collision to all links

File: src/meldog_description/description/hip/hip.urdf.xacro (robot description, xacro)
@@ -2,29 +2,30 @@
 <robot xmlns:xacro="http://www.ros.org/wiki/xacro" name = "meldog_hip">
     <xacro:property name="hip_length" value="0.2"/>
-    <xacro:property name="hip_width" value="0.1"/>
-    <xacro:property name="hip_height" value="0.05"/>
+    <xacro:property name="hip_width" value="0.15"/>
+    <xacro:property name="hip_height" value="0.075"/>
+    <xacro:property name="hip_mass" value="3.0"/>
     <xacro:macro name="hip_link" params="position">
         <link name="hip_${position}_link">
             <inertial>
-                <origin xyz="0.0 0.0 0.0" rpy="0.0 0.0 0.0"/>
-                <mass value="3.0"/>
-                <inertia ixx="1.0" ixy="1.0" ixz="1.0" iyy="1.0" iyz="1.0" izz="1.0"/>
+                <origin xyz="${hip_length/2} 0.0 0.0" rpy="0.0 0.0 0.0"/>
+                <mass value="${hip_mass}"/>
+                 <mass value="${trunk_mass}"/>
+            <inertia ixx="${1/12*trunk_mass*(hip_width*hip_width + hip_height*hip_height)}" ixy="0.0" ixz="0.0" iyy="${1/12*trunk_mass*(hip_length*hip_length + hip_height*hip_height)}" iyz=".0" izz="${1/12*trunk_mass*(hip_length*hip_length + hip_width*hip_width)}"/>
             </inertial>
-            <visual name="">
+            <visual name="hip_${position}_link_visual">
                 <origin xyz="${hip_length/2} 0.0 0.0" rpy="0.0 0.0 0.0"/>
                 <geometry>
                     <box size="${hip_length} ${hip_width} ${hip_height}"/>
                 </geometry>
-                <material name="hip_${position}_link">
+                <material name="">
                     <color rgba="1.0 0.0 0.0 1.0"/>
-                    <texture filename=""/>
                 </material>
             </visual>
-            <!-- <collision>
-                <origin xyz="0.0 0.0 0.0" rpy="0.0 0.0 0.0"/>
+            <collision name="hip_${position}_link_collision">
+                <origin xyz="${hip_length/2} 0.0 0.0" rpy="0.0 0.0 0.0"/>
                 <geometry>
-                    <box size="0.0 0.0 0.0"/>
+                    <box size="${hip_length} ${hip_width} ${hip_height}"/>
                 </geometry>
-            </collision> -->
+            </collision>
         </link>
     </xacro:macro>

File: src/meldog_description/description/shank/shank.urdf.xacro (robot description, xacro)
@@ -3,38 +3,43 @@
     <xacro:property name="shank_length" value="0.5"/>
     <xacro:property name="shank_radius" value="0.05"/>
-    <xacro:property name="feet_radius"  value ="0.08"/>
+    <xacro:property name="feet_radius" value ="0.08"/>
+    <xacro:property name="shank_mass" value = "1.0"/>
     <xacro:macro name="shank_link" params="position">
         <link name="shank_${position}_link">
             <inertial>
-                <origin xyz="0.0 0.0 0.0" rpy="0.0 0.0 0.0"/>
-                <mass value="1.0"/>
-                <inertia ixx="1.0" ixy="1.0" ixz="1.0" iyy="1.0" iyz="1.0" izz="1.0"/>
+                <origin xyz="0.0 0.0 ${-shank_length/2}" rpy="0.0 0.0 0.0"/>
+                <mass value="${shank_mass}"/>
+                <inertia ixx="${1/12*shank_mass*(3*shank_radius*shank_radius+shank_length*shank_length)}" ixy="0.0" ixz="0.0" iyy="${1/12*shank_mass*(3*shank_radius*shank_radius+shank_length*shank_length)}" iyz="0.0" izz="${1/2*shank_mass*shank_radius*shank_radius}"/>
             </inertial>
-            <visual name="">
+            <visual name="shank_${position}_link_visual">
                 <origin xyz="0.0 0.0 ${-shank_length/2}" rpy="0.0 0.0 0.0"/>
                 <geometry>
                     <cylinder radius="${shank_radius}" length="${shank_length}"/>
                 </geometry>
-                <material name="yellow">
+                <material name="">
                     <color rgba="1.0 1.0 0.0 1.0"/>
-                    <texture filename=""/>
                 </material>
             </visual>
-            <visual name="">
+            <visual name="feet_visual">
                 <origin xyz="0.0 0.0 ${-shank_length}" rpy="0.0 0.0 0.0"/>
                 <geometry>
                     <sphere radius="${feet_radius}"/>
                 </geometry>
-                <material name="purple">
+                <material name="">
                     <color rgba="1.0 0.0 1.0 1.0"/>
-                    <texture filename=""/>
                 </material>
             </visual>
-            <!-- <collision>
-                <origin xyz="0.0 0.0 0.0" rpy="0.0 0.0 0.0"/>
+            <collision name="shank_${position}_link_collision">
+                <origin xyz="0.0 0.0 ${-shank_length/2}" rpy="0.0 0.0 0.0"/>
                 <geometry>
-                    <box size="0.0 0.0 0.0"/>
+                    <cylinder radius="${shank_radius}" length="${shank_length}"/>
                 </geometry>
-            </collision> -->
+            </collision>
+            <collision name="feet_collision">
+                <origin xyz="0.0 0.0 ${-shank_length}" rpy="0.0 0.0 0.0"/>
+                <geometry>
+                    <sphere radius="${feet_radius}"/>
+                </geometry>
+            </collision>
         </link>
     </xacro:macro>

File: src/meldog_description/description/thigh/thigh.urdf.xacro (robot description, xacro)
@@ -3,27 +3,27 @@
     <xacro:property name="thigh_length" value="0.5"/>
     <xacro:property name="thigh_radius" value="0.05"/>
+    <xacro:property name="thigh_mass" value="1.0"/>
     <xacro:macro name="thigh_link" params="position">
         <link name="thigh_${position}_link">
             <inertial>
-                <origin xyz="0.0 0.0 0.0" rpy="0.0 0.0 0.0"/>
-                <mass value="1.0"/>
-                <inertia ixx="1.0" ixy="1.0" ixz="1.0" iyy="1.0" iyz="1.0" izz="1.0"/>
+                <origin xyz="0.0 0.0 ${-thigh_length/2}" rpy="0.0 0.0 0.0"/>
+                <mass value="${thigh_mass}"/>
+                <inertia ixx="${1/12*thigh_mass*(3*thigh_radius*thigh_radius+thigh_length*thigh_length)}" ixy="0.0" ixz="0.0" iyy="${1/12*thigh_mass*(3*thigh_radius*thigh_radius+thigh_length*thigh_length)}" iyz="0.0" izz="${1/2*thigh_mass*thigh_radius*thigh_radius}"/>
             </inertial>
-            <visual name="">
+            <visual name="thigh_${position}_link_visual">
                 <origin xyz="0.0 0.0 ${-thigh_length/2}" rpy="0.0 0.0 0.0"/>
                 <geometry>
                     <cylinder radius="${thigh_radius}" length="${thigh_length}"/>
                 </geometry>
-                <material name="thigh_${position}_link">
+                <material name="">
                     <color rgba="0.0 1.0 0.0 1.0"/>
-                    <texture filename=""/>
                 </material>
             </visual>
-            <!-- <collision>
-                <origin xyz="0.0 0.0 0.0" rpy="0.0 0.0 0.0"/>
+            <collision name="thigh_${position}_link_collision">
+                <origin xyz="0.0 0.0 ${-thigh_length/2}" rpy="0.0 0.0 0.0"/>
                 <geometry>
-                    <box size="0.0 0.0 0.0"/>
+                    <cylinder radius="${thigh_radius}" length="${thigh_length}"/>
                 </geometry>
-            </collision> -->
+            </collision>
         </link>
     </xacro:macro>

File: src/meldog_description/description/trunk/trunk.urdf.xacro (robot description, xacro)
@@ -7,21 +7,21 @@
     <xacro:property name="trunk_actuators_width" value="0.2" />
     <xacro:property name="trunk_actuators_height" value="0.1" />
+    <xacro:property name="trunk_mass" value="8.0"/>
     <link name="trunk_link">
         <inertial>
             <origin xyz="0.0 0.0 0.0" rpy="0.0 0.0 0.0"/>
-            <mass value="5.0"/> <!--testing-->
-            <inertia ixx="1.0" ixy="1.0" ixz="1.0" iyy="1.0" iyz="1.0" izz="1.0"/> <!--testing-->
+            <mass value="${trunk_mass}"/>
+            <inertia ixx="${1/12*trunk_mass*(trunk_base_width*trunk_base_width + trunk_base_height*trunk_base_height)}" ixy="0.0" ixz="0.0" iyy="${1/12*trunk_mass*(trunk_base_length*trunk_base_length + trunk_base_height*trunk_base_height)}" iyz=".0" izz="${1/12*trunk_mass*(trunk_base_length*trunk_base_length + trunk_base_width*trunk_base_width)}"/>
         </inertial>
-        <visual name="trunk_base">
+        <visual name="trunk_base_visual">
             <origin xyz="0.0 0.0 0.0" rpy="0.0 0.0 0.0"/>
             <geometry>
                 <box size="${trunk_base_length} ${trunk_base_width} ${trunk_base_height}"/>
             </geometry>
-            <material name="trunk_base_color">
+            <material name="">
                 <color rgba="0.0 0.0 1.0 1.0"/>
-                <texture filename=""/>
             </material>
         </visual>
-        <visual name="trunk_actuators_left">
+        <visual name="trunk_actuators_left_visual">
             <origin xyz="0.0 ${trunk_base_width/2 + trunk_actuators_width/2} 0.0" rpy="0.0 0.0 0.0"/>
             <geometry>
@@ -30,8 +30,7 @@
             <material name="">
                 <color rgba="0.0 1.0 0.0 1.0"/>
-                <texture filename="trunk_actuators_left_color"/>
             </material>
         </visual>
-        <visual name="trunk_actuators_right">
+        <visual name="trunk_actuators_right_visual">
             <origin xyz="0.0 ${-trunk_base_width/2 - trunk_actuators_width/2} 0.0" rpy="0.0 0.0 0.0"/>
             <geometry>
@@ -40,11 +39,22 @@
             <material name="">
                 <color rgba="1.0 0.0 0.0 1.0"/>
-                <texture filename="trunk_actuators_right_color"/>
             </material>
         </visual>
-        <collision> <!--testing-->
+         <collision name="trunk_base_collision">
             <origin xyz="0.0 0.0 0.0" rpy="0.0 0.0 0.0"/>
             <geometry>
-                <box size="1.0 1.0 1.0"/>
+                <box size="${trunk_base_length} ${trunk_base_width} ${trunk_base_height}"/>
+            </geometry>
+        </collision>
+        <collision name="trunk_actuators_left_collision">
+            <origin xyz="0.0 ${trunk_base_width/2 + trunk_actuators_width/2} 0.0" rpy="0.0 0.0 0.0"/>
+            <geometry>
+                <box size="${trunk_actuators_length} ${trunk_actuators_width} ${trunk_actuators_height}"/>
+            </geometry>
+        </collision>
+        <collision name="trunk_actuators_right_collision">
+            <origin xyz="0.0 ${-trunk_base_width/2 - trunk_actuators_width/2} 0.0" rpy="0.0 0.0 0.0"/>
+            <geometry>
+                <box size="${trunk_actuators_length} ${trunk_actuators_width} ${trunk_actuators_height}"/>
             </geometry>
         </collision>
