Commit message: Added feet links and joints, added realistic joint limits for actuators

File: src/meldog_description/description/common/actuator_macros.urdf.xacro (robot description, xacro)
@@ -1,8 +1,8 @@
 <?xml version="1.0"?>
 <robot xmlns:xacro="http://www.ros.org/wiki/xacro" name = "meldog_actuator">
-    <xacro:property name="actuator_max_velocity" value="0.5"/>
-    <xacro:property name="actuator_max_torque" value="0.5"/>
-    <xacro:property name="actuator_damping" value="0.5"/>
-    <xacro:property name="actuator_friction" value="1.788"/>
+    <xacro:property name="actuator_max_velocity" value="20.2"/>
+    <xacro:property name="actuator_max_torque" value="30"/>
+    <xacro:property name="actuator_damping" value="0.0"/>
+    <xacro:property name="actuator_friction" value="0.0"/>
     <xacro:macro name ="meldog_joint_limits" params="lower upper">
         <limit lower="${lower}" upper="${upper}" effort="${actuator_max_torque}" velocity="${actuator_max_velocity}"/>

File: src/meldog_description/description/common/gazebo_macros.urdf.xacro (robot description, xacro)
@@ -8,6 +8,5 @@
     <xacro:property name="maxVel_value" value="0.1"/>
     <xacro:property name="dampingFactor_value" value="0.004"/>
-    <xacro:property name="selfCollide_value" value="false"/>
-    <xacro:macro name="gazebo_link" params="link_name color">
+    <xacro:macro name="gazebo_link" params="link_name color selfCollide_value">
         <gazebo reference="${link_name}">
             <material>Gazebo/${color}</material>

File: src/meldog_description/description/meldog_core.urdf.xacro (robot description, xacro)
@@ -1,6 +1,8 @@
 <?xml version="1.0"?>
-<robot xmlns:xacro="http://www.ros.org/wiki/xacro" name = "meldog_core">
+<robot xmlns:xacro="http://www.ros.org/wiki/xacro" name="meldog_core">
     <!-- PI -->
     <xacro:property name="PI" value="3.1415926535897"/>
+    <!-- Actuator macros -->
+    <xacro:include filename="common/actuator_macros.urdf.xacro"/>
     <!-- LINKS: -->
     <!-- Base link spawns in x= 0.0 y = 0.0 z = 0.0 -->
@@ -27,8 +29,9 @@
     <xacro:shank_link position="back_right"/>
     <!-- Feet links (frames in the end of shank) -->
-    <link name="feet_front_left_link"></link>
-    <link name="feet_front_right_link"></link>
-    <link name="feet_back_left_link"></link>
-    <link name="feet_back_right_link"></link>
+    <xacro:include filename="feet/feet.urdf.xacro"/>
+    <xacro:feet_link position="front_left"/>
+    <xacro:feet_link position="front_right"/>
+    <xacro:feet_link position="back_left"/>
+    <xacro:feet_link position="back_right"/>
     <!-- JOINTS: -->
     <!-- Base to Trunk joint -->
@@ -45,5 +48,5 @@
         <child link="hip_front_left_link"/>
         <axis xyz="1.0 0.0 0.0"/>
-        <limit lower="-1.0" upper="1" effort="10.0" velocity="100.0"/>
+        <xacro:meldog_joint_limits lower ="-${PI/2}" upper = "${PI/2}"/>
     </joint>
     <!-- Trunk to Hip front right joint -->
@@ -53,5 +56,5 @@
         <child link="hip_front_right_link"/>
         <axis xyz="-1.0 0.0 0.0"/>
-        <limit lower="-1.0" upper="1" effort="10.0" velocity="100.0"/>
+        <xacro:meldog_joint_limits lower ="-${PI/2}" upper = "${PI/2}"/>
     </joint>
     <!-- Trunk to Hip back left joint -->
@@ -61,5 +64,5 @@
         <child link="hip_back_left_link"/>
         <axis xyz="-1.0 0.0 0.0"/>
-        <limit lower="-1.0" upper="1" effort="10.0" velocity="100.0"/>
+        <xacro:meldog_joint_limits lower ="-${PI/2}" upper = "${PI/2}"/>
     </joint>
     <!-- Trunk to Hip back right joint -->
@@ -69,5 +72,5 @@
         <child link="hip_back_right_link"/>
         <axis xyz="1.0 0.0 0.0"/>
-        <limit lower="-1.0" upper="1" effort="10.0" velocity="100.0"/>
+        <xacro:meldog_joint_limits lower ="-${PI/2}" upper = "${PI/2}"/>
     </joint>
     <!-- Hip front left to Thigh front left -->
@@ -77,5 +80,5 @@
         <child link="thigh_front_left_link"/>
         <axis xyz="0.0 -1.0 0.0"/>
-        <limit lower="-1.0" upper="1.0" effort="10.0" velocity="100.0"/>
+        <xacro:meldog_joint_limits lower ="-${PI}" upper = "${PI}"/>
     </joint>
     <!-- Hip front right to Thigh front right -->
@@ -85,5 +88,5 @@
         <child link="thigh_front_right_link"/>
         <axis xyz="0.0 -1.0 0.0"/>
-        <limit lower="-1.0" upper="1.0" effort="10.0" velocity="100.0"/>
+        <xacro:meldog_joint_limits lower ="-${PI}" upper = "${PI}"/>
     </joint>
     <!-- Hip back left to Thigh back left -->
@@ -93,5 +96,5 @@
         <child link="thigh_back_left_link"/>
         <axis xyz="0.0 1.0 0.0"/>
-        <limit lower="-1.0" upper="1.0" effort="10.0" velocity="100.0"/>
+        <xacro:meldog_joint_limits lower ="-${PI}" upper = "${PI}"/>
     </joint>
     <!-- Hip back right to Thigh back right -->
@@ -101,5 +104,5 @@
         <child link="thigh_back_right_link"/>
         <axis xyz="0.0 1.0 0.0"/>
-        <limit lower="-1.0" upper="1.0" effort="10.0" velocity="100.0"/>
+        <xacro:meldog_joint_limits lower ="-${PI}" upper = "${PI}"/>
     </joint>
     <!-- Thigh front left to Shank front left -->
@@ -109,5 +112,5 @@
         <child link="shank_front_left_link"/>
         <axis xyz="0.0 -1.0 0.0"/>
-        <limit lower="-1.0" upper="1.0" effort="10.0" velocity="100.0"/>
+        <xacro:meldog_joint_limits lower ="-${PI/2}" upper = "${PI/2}"/>
     </joint>
     <!-- Thigh front right to Shank front right -->
@@ -117,5 +120,5 @@
         <child link="shank_front_right_link"/>
         <axis xyz="0.0 -1.0 0.0"/>
-        <limit lower="-1.0" upper="1.0" effort="10.0" velocity="100.0"/>
+        <xacro:meldog_joint_limits lower ="-${PI/2}" upper = "${PI/2}"/>
     </joint>
     <!-- Thigh back left to Shank back left -->
@@ -125,5 +128,5 @@
         <child link="shank_back_left_link"/>
         <axis xyz="0.0 1.0 0.0"/>
-        <limit lower="-1.0" upper="1.0" effort="10.0" velocity="100.0"/>
+        <xacro:meldog_joint_limits lower ="-${PI/2}" upper = "${PI/2}"/>
     </joint>
     <!-- Thigh back right to Shank back right -->
@@ -133,5 +136,5 @@
         <child link="shank_back_right_link"/>
         <axis xyz="0.0 1.0 0.0"/>
-        <limit lower="-1.0" upper="1.0" effort="10.0" velocity="100.0"/>
+        <xacro:meldog_joint_limits lower ="-${PI/2}" upper = "${PI/2}"/>
     </joint>
     <!-- Shank front left to Feet front left -->

File: src/meldog_description/description/shank/shank.urdf.xacro (robot description, xacro)
@@ -3,5 +3,4 @@
     <xacro:property name="shank_length" value="0.5"/>
     <xacro:property name="shank_radius" value="0.05"/>
-    <xacro:property name="feet_radius" value ="0.08"/>
     <xacro:property name="shank_mass" value = "1.0"/>
     <xacro:macro name="shank_link" params="position">
@@ -21,13 +20,4 @@
                 </material>
             </visual>
-            <visual name="feet_visual">
-                <origin xyz="0.0 0.0 ${-shank_length}" rpy="0.0 0.0 0.0"/>
-                <geometry>
-                    <sphere radius="${feet_radius}"/>
-                </geometry>
-                <material name="">
-                    <color rgba="1.0 0.0 1.0 1.0"/>
-                </material>
-            </visual>
             <collision name="shank_${position}_link_collision">
                 <origin xyz="0.0 0.0 ${-shank_length/2}" rpy="0.0 0.0 0.0"/>
@@ -36,10 +26,4 @@
                 </geometry>
             </collision>
-            <collision name="feet_collision">
-                <origin xyz="0.0 0.0 ${-shank_length}" rpy="0.0 0.0 0.0"/>
-                <geometry>
-                    <sphere radius="${feet_radius}"/>
-                </geometry>
-            </collision>
         </link>
     </xacro:macro>
