Commit message: Succesfully run meldog urdf in gazebo classic

File: src/meldog_description/description/gazebo/gazebo_macros.urdf.xacro (robot description, xacro)
@@ -3,31 +3,31 @@
     <!-- Gazebo macro for links -->
     <xacro:property name="kp_value" value="25000.0"/>
-    <xacro:property name="kd_value" value="0.05"/>
-    <xacro:property name="mu2_value" value="50"/>
-    <xacro:property name="mu2_value" value="25"/>
-    <xacro:property name="maxVel_value" value="0.1"/>
-    <xacro:property name="dampingFactor_value" value="0.004"/>
+    <xacro:property name="kd_value" value="0.15"/>
+    <xacro:property name="mu2_value" value="0.7"/>
+    <xacro:property name="mu2_value" value="0.7"/>
+    <xacro:property name="maxVel_value" value="0.25"/>
+    <xacro:property name="dampingFactor_value" value="0.00"/>
     <xacro:macro name="gazebo_link" params="link_name color selfCollide_value">
         <gazebo reference="${link_name}_link">
             <material>Gazebo/${color}</material>
-              <mu1 value="${mu2_value}"/>
-              <mu2 value="${mu2_value}"/>
-              <kp value="${kp_value}" />
-              <kd value="${kd_value}" />
-              <maxVel value="${maxVel_value}"/>
-              <dampingFactor value="${dampingFactor_value}"/>
-              <selfCollide>${selfCollide_value}</selfCollide>
+            <mu1 value="${mu2_value}"/>
+            <mu2 value="${mu2_value}"/>
+            <kp value="${kp_value}" />
+            <kd value="${kd_value}" />
+            <maxVel value="${maxVel_value}"/>
+            <dampingFactor value="${dampingFactor_value}"/>
+            <selfCollide value="${selfCollide_value}"/>
         </gazebo>
     </xacro:macro>
     <!-- Gazebo macro for joints -->
-    <xacro:property name="damper_value" value="true"/>
-    <xacro:property name="springStiffness_value" value="0.5"/>
-    <xacro:property name="springReference_value" value="0.061"/>
-    <xacro:property name="stopErp_value" value="0.2"/>
-    <xacro:property name="stopCfm_value" value="0.45"/>
+    <xacro:property name="implicitSpringDamper_value" value="true"/>
+    <xacro:property name="springStiffness_value" value="0.0"/>
+    <xacro:property name="springReference_value" value="0.0"/>
+    <xacro:property name="stopErp_value" value="0.0"/>
+    <xacro:property name="stopCfm_value" value="0.0"/>
     <xacro:macro name="gazebo_joint" params="joint_name">
-        <gazebo reference="${joint_name_joint}">
-            <implicitSpringDamper>${Damper_value}</implicitSpringDamper>
-            <springStiffness>${springstiffness_value}</springStiffness>
+        <gazebo reference="${joint_name}_joint">
+            <implicitSpringDamper>${implicitSpringDamper_value}</implicitSpringDamper>
+            <springStiffness>${springStiffness_value}</springStiffness>
             <springReference>${springReference_value}</springReference>
             <stopErp>${stopErp_value}</stopErp>

File: src/meldog_description/description/meldog_gazebo.urdf.xacro (robot description, xacro)
@@ -1,29 +1,31 @@
 <?xml version="1.0"?>
 <robot xmlns:xacro="http://www.ros.org/wiki/xacro" name = "meldog_gazebo">
+    <!-- Meldog Core file -->
+    <xacro:include filename="meldog_core.urdf.xacro"/>
     <!-- Gazebo macros -->
     <xacro:include filename="gazebo/gazebo_macros.urdf.xacro"/>
     <!-- LINKS: -->
     <!-- Trunk link -->
-    <xacro:gazebo_link link_name="trunk" color="Blue" selfCollide_value ="false"/>
+    <xacro:gazebo_link link_name="trunk" color="Blue" selfCollide_value ="true"/>
     <!-- Hip links -->
-    <xacro:gazebo_link link_name="hip_front_left" color="Red" selfCollide_value ="false"/>
-    <xacro:gazebo_link link_name="hip_front_right" color="Red" selfCollide_value ="false"/>
-    <xacro:gazebo_link link_name="hip_back_left" color="Red" selfCollide_value ="false"/>
-    <xacro:gazebo_link link_name="hip_back_right" color="Red" selfCollide_value ="false"/>
+    <xacro:gazebo_link link_name="hip_front_left" color="Red" selfCollide_value ="true"/>
+    <xacro:gazebo_link link_name="hip_front_right" color="Red" selfCollide_value ="true"/>
+    <xacro:gazebo_link link_name="hip_back_left" color="Red" selfCollide_value ="true"/>
+    <xacro:gazebo_link link_name="hip_back_right" color="Red" selfCollide_value ="true"/>
     <!-- Thigh links -->
-    <xacro:gazebo_link link_name="thigh_front_left" color="Green" selfCollide_value ="false"/>
-    <xacro:gazebo_link link_name="thigh_front_right" color="Green" selfCollide_value ="false"/>
-    <xacro:gazebo_link link_name="thigh_back_left" color="Green" selfCollide_value ="false"/>
-    <xacro:gazebo_link link_name="thigh_back_right" color="Green" selfCollide_value ="false"/>
+    <xacro:gazebo_link link_name="thigh_front_left" color="Green" selfCollide_value ="true"/>
+    <xacro:gazebo_link link_name="thigh_front_right" color="Green" selfCollide_value ="true"/>
+    <xacro:gazebo_link link_name="thigh_back_left" color="Green" selfCollide_value ="true"/>
+    <xacro:gazebo_link link_name="thigh_back_right" color="Green" selfCollide_value ="true"/>
     <!-- Shank links -->
-    <xacro:gazebo_link link_name="shank_front_left_" color="Yellow" selfCollide_value ="false"/>
-    <xacro:gazebo_link link_name="shank_front_right" color="Yellow" selfCollide_value ="false"/>
-    <xacro:gazebo_link link_name="shank_back_left" color="Yellow" selfCollide_value ="false"/>
-    <xacro:gazebo_link link_name="shank_back_right" color="Yellow" selfCollide_value ="false"/>
+    <xacro:gazebo_link link_name="shank_front_left_" color="Yellow" selfCollide_value ="true"/>
+    <xacro:gazebo_link link_name="shank_front_right" color="Yellow" selfCollide_value ="true"/>
+    <xacro:gazebo_link link_name="shank_back_left" color="Yellow" selfCollide_value ="true"/>
+    <xacro:gazebo_link link_name="shank_back_right" color="Yellow" selfCollide_value ="true"/>
     <!-- Feet links -->
-    <xacro:gazebo_link link_name="feet_front_left" color="Pink" selfCollide_value ="false"/>
-    <xacro:gazebo_link link_name="feet_front_right" color="Pink" selfCollide_value ="false"/>
-    <xacro:gazebo_link link_name="feet_back_left" color="Pink" selfCollide_value ="false"/>
-    <xacro:gazebo_link link_name="feet_back_right" color="Pink" selfCollide_value ="false"/>
+    <xacro:gazebo_link link_name="feet_front_left" color="Pink" selfCollide_value ="true"/>
+    <xacro:gazebo_link link_name="feet_front_right" color="Pink" selfCollide_value ="true"/>
+    <xacro:gazebo_link link_name="feet_back_left" color="Pink" selfCollide_value ="true"/>
+    <xacro:gazebo_link link_name="feet_back_right" color="Pink" selfCollide_value ="true"/>
     <!-- JOINTS (only revolute): -->
     <!-- Trunk to Hips joints-->

File: src/meldog_description/description/meldog_links/shank/shank.urdf.xacro (robot description, xacro)
@@ -23,5 +23,5 @@
                 <origin xyz="0.0 0.0 ${-shank_length/2}" rpy="0.0 0.0 0.0"/>
                 <geometry>
-                    <cylinder radius="${shank_radius}" length="${shank_length}"/>
+                    <cylinder radius="${shank_radius}" length="${3*shank_length/4}"/>
                 </geometry>
             </collision>

File: src/meldog_description/description/meldog_links/thigh/thigh.urdf.xacro (robot description, xacro)
@@ -23,5 +23,5 @@
                 <origin xyz="0.0 0.0 ${-thigh_length/2}" rpy="0.0 0.0 0.0"/>
                 <geometry>
-                    <cylinder radius="${thigh_radius}" length="${thigh_length}"/>
+                    <cylinder radius="${thigh_radius}" length="${3*thigh_length/4}"/>
                 </geometry>
             </collision>
