Commit message: Succesfully runned simulation with ros2 control plugin and controllers

File: src/meldog_simple_description/description/meldog_gazebo.urdf.xacro (robot description, xacro)
@@ -44,3 +44,5 @@
     <xacro:gazebo_joint joint_name="BLS"/>
     <xacro:gazebo_joint joint_name="BRS"/>
+    <!-- ROS2 Control -->
+    <xacro:include filename="ros2_control/ros2_control_gazebo.urdf.xacro"/>
 </robot>

File: src/meldog_simple_description/description/ros2_control/ros2_control_gazebo.urdf.xacro (robot description, xacro)
@@ -7,22 +7,22 @@
         </hardware>
         <!-- Transmissions -->
-        <xacro:include filename="ros2_control/transmission_macros.urdf.xacro"/>
+        <!-- <xacro:include filename="transmission_macros.urdf.xacro"/> -->
         <!-- Hardware interface for Gazebo -->
-        <xacro:include filename="ros2_control/ros2_control_joint_macros.urdf.xacro"/>
+        <xacro:include filename="ros2_control_joint_macros.urdf.xacro"/>
         <!-- Trunk to Hips joints-->
-        <xacro:ros2_control_joint joint_name="FLH_joint" lower="-${PI/2}" upper="${PI/2}"/>
-        <xacro:ros2_control_joint joint_name="FRH_joint" lower="-${PI/2}" upper="${PI/2}"/>
-        <xacro:ros2_control_joint joint_name="BLH_joint" lower="-${PI/2}" upper="${PI/2}"/>
-        <xacro:ros2_control_joint joint_name="BRH_joint" lower="-${PI/2}" upper="${PI/2}"/>
+        <xacro:ros2_control_joint joint_name="FLH" lower="-${PI/2}" upper="${PI/2}"/>
+        <xacro:ros2_control_joint joint_name="FRH" lower="-${PI/2}" upper="${PI/2}"/>
+        <xacro:ros2_control_joint joint_name="BLH" lower="-${PI/2}" upper="${PI/2}"/>
+        <xacro:ros2_control_joint joint_name="BRH" lower="-${PI/2}" upper="${PI/2}"/>
         <!-- Hips to Thighs joints -->
-        <xacro:ros2_control_joint joint_name="FLT_joint" lower="-${PI}" upper="${PI}"/>
-        <xacro:ros2_control_joint joint_name="FRT_joint" lower="-${PI}" upper="${PI}"/>
-        <xacro:ros2_control_joint joint_name="BLT_joint" lower="-${PI}" upper="${PI}"/>
-        <xacro:ros2_control_joint joint_name="BRT_joint" lower="-${PI}" upper="${PI}"/>
+        <xacro:ros2_control_joint joint_name="FLT" lower="-${PI}" upper="${PI}"/>
+        <xacro:ros2_control_joint joint_name="FRT" lower="-${PI}" upper="${PI}"/>
+        <xacro:ros2_control_joint joint_name="BLT" lower="-${PI}" upper="${PI}"/>
+        <xacro:ros2_control_joint joint_name="BRT" lower="-${PI}" upper="${PI}"/>
         <!-- Thighs to Shanks joints -->
-        <xacro:ros2_control_joint joint_name="FLS_joint" lower="-${PI/2}" upper="${PI/2}"/>
-        <xacro:ros2_control_joint joint_name="FRS_joint" lower="-${PI/2}" upper="${PI/2}"/>
-        <xacro:ros2_control_joint joint_name="BLS_joint" lower="-${PI/2}" upper="${PI/2}"/>
-        <xacro:ros2_control_joint joint_name="BRS_joint" lower="-${PI/2}" upper="${PI/2}"/>
+        <xacro:ros2_control_joint joint_name="FLS" lower="-${PI/2}" upper="${PI/2}"/>
+        <xacro:ros2_control_joint joint_name="FRS" lower="-${PI/2}" upper="${PI/2}"/>
+        <xacro:ros2_control_joint joint_name="BLS" lower="-${PI/2}" upper="${PI/2}"/>
+        <xacro:ros2_control_joint joint_name="BRS" lower="-${PI/2}" upper="${PI/2}"/>
     </ros2_control>
     <gazebo>

File: src/meldog_simple_description/description/ros2_control/ros2_control_joint_macros.urdf.xacro (robot description, xacro)
@@ -1,6 +1,6 @@
 <?xml version="1.0"?>
 <robot xmlns:xacro="http://www.ros.org/wiki/xacro" name ="meldog_ros2_control_joint_macros">
-    <xacro:include filename="actuator/actuator_macros.urdf.xacro"/>
-    <xacro:macro name="ros2_control_joint" params="joint_name upper lower"/>
+    <xacro:include filename="../actuator/actuator_macros.urdf.xacro"/>
+    <xacro:macro name="ros2_control_joint" params="joint_name upper lower">
         <joint name="${joint_name}_joint">
             <command_interface name="position">
@@ -12,9 +12,8 @@
                 <param name="max">${actuator_max_velocity}</param>
             </command_interface>
-            <xacro:if value="$(arg use_gazebo)">
-                <command_interface name="effort"/>
-                    <param name="min">-${actuator_max_torque}</param>
-                    <param name="max">${actuator_max_torque}</param>
-            </xacro:if>
+            <command_interface name="effort">
+                <param name="min">-${actuator_max_torque}</param>
+                <param name="max">${actuator_max_torque}</param>
+            </command_interface>
             <state_interface name="position"/>
             <state_interface name="velocity"/>

File: src/meldog_simple_description/description/ros2_control/transmission_macros.urdf.xacro (robot description, xacro)
@@ -2,5 +2,5 @@
 <robot xmlns:xacro="http://www.ros.org/wiki/xacro" name ="meldog_transmissions">
     <!-- SimpleTransmission macro -->
-    <xacro:macro name="SimpleTransmission" params="joint_name reduction offset"/>
+    <xacro:macro name="SimpleTransmission" params="joint_name reduction offset">
         <transmission name="SimpleTransmission_${joint_name}">
                 <plugin>transmission_interface/SimpleTransmission</plugin>
@@ -13,6 +13,6 @@
     </xacro:macro>
     <!-- FourBarLinkageTransmission macro -->
-    <xacro:macro name="FourBarLinkageTransmission" params="first_joint_name second__joint_name reduction first_offset second_offset"/>
-        <transmission name="FourBarLinkageTransmission_${first_joint_name}_${second__joint_name}">
+    <xacro:macro name="FourBarLinkageTransmission" params="first_joint_name second_joint_name reduction first_offset second_offset">
+        <transmission name="FourBarLinkageTransmission_${first_joint_name}_${second_joint_name}">
             <plugin>transmission_interface/FourBarLinkageTransmission</plugin>
             <actuator name="${first_joint_name}_actuator" role="actuator1">
@@ -39,7 +39,7 @@
     <xacro:SimpleTransmission joint_name="BRH" reduction="9.97" offset="0.0"/>
     <!-- Thighs to Shanks transmissions -->
-    <xacro:FourBarLinkageTransmission first_joint_name="FLT" second__joint_name="FLS" reduction="9.97" first_offset="0.0" second_offset="0.0"/>
-    <xacro:FourBarLinkageTransmission first_joint_name="FRT" second__joint_name="FRS" reduction="9.97" first_offset="0.0" second_offset="0.0"/>
-    <xacro:FourBarLinkageTransmission first_joint_name="BLT" second__joint_name="BLS" reduction="9.97" first_offset="0.0" second_offset="0.0"/>
-    <xacro:FourBarLinkageTransmission first_joint_name="BRT" second__joint_name="BRS" reduction="9.97" first_offset="0.0" second_offset="0.0"/>
+    <xacro:FourBarLinkageTransmission first_joint_name="FLT" second_joint_name="FLS" reduction="9.97" first_offset="0.0" second_offset="0.0"/>
+    <xacro:FourBarLinkageTransmission first_joint_name="FRT" second_joint_name="FRS" reduction="9.97" first_offset="0.0" second_offset="0.0"/>
+    <xacro:FourBarLinkageTransmission first_joint_name="BLT" second_joint_name="BLS" reduction="9.97" first_offset="0.0" second_offset="0.0"/>
+    <xacro:FourBarLinkageTransmission first_joint_name="BRT" second_joint_name="BRS" reduction="9.97" first_offset="0.0" second_offset="0.0"/>
 </robot>
