Commit message: Cleaned up code, added new macros and properties

File: src/meldog_simple_description/description/meldog_core.urdf.xacro (robot description, xacro)
@@ -3,13 +3,14 @@
     <!-- PI -->
     <xacro:property name="PI" value="3.1415926535897"/>
-    <!-- Actuator macros -->
-    <xacro:include filename="actuator/actuator_macros.urdf.xacro"/>
+    <!-- Joint properties and macros: -->
+    <xacro:include filename="joints/joint_properties.urdf.xacro"/>
+    <xacro:include filename="joints/joint_macros.urdf.xacro"/>
     <!-- LINKS: -->
     <!-- Base link spawns in x= 0.0 y = 0.0 z = 0.0 -->
     <link name="base_link"></link>
     <!-- Trunk link -->
-    <xacro:include filename="meldog_links/trunk/trunk.urdf.xacro"/>
+    <xacro:include filename="links/trunk/trunk.urdf.xacro"/>
     <!-- Hip links -->
-    <xacro:include filename="meldog_links/hip/hip.urdf.xacro"/>
+    <xacro:include filename="links/hip/hip.urdf.xacro"/>
     <xacro:hip_link position="front_left"/>
     <xacro:hip_link position="front_right"/>
@@ -17,5 +18,5 @@
     <xacro:hip_link position="back_right"/>
     <!-- Thigh links -->
-    <xacro:include filename="meldog_links/thigh/thigh.urdf.xacro"/>
+    <xacro:include filename="links/thigh/thigh.urdf.xacro"/>
     <xacro:thigh_link position="front_left"/>
     <xacro:thigh_link position="front_right"/>
@@ -23,5 +24,5 @@
     <xacro:thigh_link position="back_right"/>
     <!-- Shank links -->
-    <xacro:include filename="meldog_links/shank/shank.urdf.xacro"/>
+    <xacro:include filename="links/shank/shank.urdf.xacro"/>
     <xacro:shank_link position="front_left"/>
     <xacro:shank_link position="front_right"/>
@@ -29,5 +30,5 @@
     <xacro:shank_link position="back_right"/>
     <!-- Feet links (frames in the end of shank) -->
-    <xacro:include filename="meldog_links/feet/feet.urdf.xacro"/>
+    <xacro:include filename="links/feet/feet.urdf.xacro"/>
     <xacro:feet_link position="front_left"/>
     <xacro:feet_link position="front_right"/>
@@ -39,6 +40,5 @@
         <parent link="base_link"/>
         <child link="trunk_link"/>
-        <!--Origin defines translation child frame relative to parent frame. Translation is performed in parent frame.-->
-        <origin xyz="0 0 1.0" rpy="0 0 0"/>  <!--testing-->
+        <origin xyz="0 0 1.0" rpy="0 0 0"/>
     </joint>
     <!-- Trunk to Hip front left joint -->
@@ -48,5 +48,5 @@
         <child link="hip_front_left_link"/>
         <axis xyz="1.0 0.0 0.0"/>
-        <xacro:meldog_joint_limits lower ="-${PI/2}" upper = "${PI/2}"/>
+        <xacro:joint_macro lower ="${H_lower_limit}" upper = "${H_upper_limit}"/>
     </joint>
     <!-- Trunk to Hip front right joint -->
@@ -56,5 +56,5 @@
         <child link="hip_front_right_link"/>
         <axis xyz="-1.0 0.0 0.0"/>
-        <xacro:meldog_joint_limits lower ="-${PI/2}" upper = "${PI/2}"/>
+        <xacro:joint_macro lower ="${H_lower_limit}" upper = "${H_upper_limit}"/>
     </joint>
     <!-- Trunk to Hip back left joint -->
@@ -64,5 +64,5 @@
         <child link="hip_back_left_link"/>
         <axis xyz="-1.0 0.0 0.0"/>
-        <xacro:meldog_joint_limits lower ="-${PI/2}" upper = "${PI/2}"/>
+        <xacro:joint_macro lower ="${H_lower_limit}" upper = "${H_upper_limit}"/>
     </joint>
     <!-- Trunk to Hip back right joint -->
@@ -72,5 +72,5 @@
         <child link="hip_back_right_link"/>
         <axis xyz="1.0 0.0 0.0"/>
-        <xacro:meldog_joint_limits lower ="-${PI/2}" upper = "${PI/2}"/>
+        <xacro:joint_macro lower ="${H_lower_limit}" upper = "${H_upper_limit}"/>
     </joint>
     <!-- Hip front left to Thigh front left -->
@@ -80,5 +80,5 @@
         <child link="thigh_front_left_link"/>
         <axis xyz="0.0 -1.0 0.0"/>
-        <xacro:meldog_joint_limits lower ="-${PI}" upper = "${PI}"/>
+        <xacro:joint_macro lower ="${T_lower_limit}" upper = "${T_upper_limit}"/>
     </joint>
     <!-- Hip front right to Thigh front right -->
@@ -88,5 +88,5 @@
         <child link="thigh_front_right_link"/>
         <axis xyz="0.0 -1.0 0.0"/>
-        <xacro:meldog_joint_limits lower ="-${PI}" upper = "${PI}"/>
+        <xacro:joint_macro lower ="${T_lower_limit}" upper = "${T_upper_limit}"/>
     </joint>
     <!-- Hip back left to Thigh back left -->
@@ -96,5 +96,5 @@
         <child link="thigh_back_left_link"/>
         <axis xyz="0.0 1.0 0.0"/>
-        <xacro:meldog_joint_limits lower ="-${PI}" upper = "${PI}"/>
+        <xacro:joint_macro lower ="${T_lower_limit}" upper = "${T_upper_limit}"/>
     </joint>
     <!-- Hip back right to Thigh back right -->
@@ -104,5 +104,5 @@
         <child link="thigh_back_right_link"/>
         <axis xyz="0.0 1.0 0.0"/>
-        <xacro:meldog_joint_limits lower ="-${PI}" upper = "${PI}"/>
+        <xacro:joint_macro lower ="${T_lower_limit}" upper = "${T_upper_limit}"/>
     </joint>
     <!-- Thigh front left to Shank front left -->
@@ -112,5 +112,5 @@
         <child link="shank_front_left_link"/>
         <axis xyz="0.0 -1.0 0.0"/>
-        <xacro:meldog_joint_limits lower ="-${5*PI/6}" upper = "${5*PI/6}"/>
+        <xacro:joint_macro lower ="${S_lower_limit}" upper = "${S_upper_limit}"/>
     </joint>
     <!-- Thigh front right to Shank front right -->
@@ -120,5 +120,5 @@
         <child link="shank_front_right_link"/>
         <axis xyz="0.0 -1.0 0.0"/>
-        <xacro:meldog_joint_limits lower ="-${5*PI/6}" upper = "${5*PI/6}"/>
+        <xacro:joint_macro lower ="${S_lower_limit}" upper = "${S_upper_limit}"/>
     </joint>
     <!-- Thigh back left to Shank back left -->
@@ -128,5 +128,5 @@
         <child link="shank_back_left_link"/>
         <axis xyz="0.0 1.0 0.0"/>
-        <xacro:meldog_joint_limits lower ="-${5*PI/6}" upper = "${5*PI/6}"/>
+        <xacro:joint_macro lower ="${S_lower_limit}" upper = "${S_upper_limit}"/>
     </joint>
     <!-- Thigh back right to Shank back right -->
@@ -136,5 +136,5 @@
         <child link="shank_back_right_link"/>
         <axis xyz="0.0 1.0 0.0"/>
-        <xacro:meldog_joint_limits lower ="-${5*PI/6}" upper = "${5*PI/6}"/>
+        <xacro:joint_macro lower ="${S_lower_limit}" upper = "${S_upper_limit}"/>
     </joint>
     <!-- Shank front left to Feet front left -->

File: src/meldog_simple_description/description/ros2_control/joints_hardware/joint_hardware_macros.urdf.xacro (robot description, xacro)
@@ -1,6 +1,5 @@
 <?xml version="1.0"?>
-<robot xmlns:xacro="http://www.ros.org/wiki/xacro" name ="meldog_ros2_control_joint_macros">
-    <xacro:include filename="../actuator/actuator_macros.urdf.xacro"/>
-    <xacro:macro name="ros2_control_joint" params="joint_name upper lower">
+<robot xmlns:xacro="http://www.ros.org/wiki/xacro" name ="joint_hardware_macros">
+    <xacro:macro name="joint_hardware_macro" params="joint_name upper lower">
         <joint name="${joint_name}_joint">
             <command_interface name="position">
@@ -9,10 +8,10 @@
             </command_interface>
             <command_interface name="velocity">
-                <param name="min">-${actuator_max_velocity}</param>
-                <param name="max">${actuator_max_velocity}</param>
+                <param name="min">-${motor_max_velocity}</param>
+                <param name="max">${motor_max_velocity}</param>
             </command_interface>
             <command_interface name="effort">
-                <param name="min">-${actuator_max_torque}</param>
-                <param name="max">${actuator_max_torque}</param>
+                <param name="min">-${motor_max_torque}</param>
+                <param name="max">${motor_max_torque}</param>
             </command_interface>
             <state_interface name="position"/>

File: src/meldog_simple_description/description/ros2_control/ros2_control_gazebo.urdf.xacro (robot description, xacro)
@@ -1,28 +1,11 @@
 <?xml version="1.0"?>
 <robot xmlns:xacro="http://www.ros.org/wiki/xacro" name = "meldog_ros2_control_gazebo">
-<!-- ROS2 Control Gazebo -->
+    <!-- ROS2 Control for Gazebo: -->
     <ros2_control name="meldog_gazebo" type="system">
         <hardware>
             <plugin>ign_ros2_control/IgnitionSystem</plugin>
         </hardware>
-        <!-- Transmissions -->
-        <!-- <xacro:include filename="transmission_macros.urdf.xacro"/> -->
-        <!-- Hardware interface for Gazebo -->
-        <xacro:include filename="ros2_control_joint_macros.urdf.xacro"/>
-        <!-- Trunk to Hips joints-->
-        <xacro:ros2_control_joint joint_name="FLH" lower="-${PI/2}" upper="${PI/2}"/>
-        <xacro:ros2_control_joint joint_name="FRH" lower="-${PI/2}" upper="${PI/2}"/>
-        <xacro:ros2_control_joint joint_name="BLH" lower="-${PI/2}" upper="${PI/2}"/>
-        <xacro:ros2_control_joint joint_name="BRH" lower="-${PI/2}" upper="${PI/2}"/>
-        <!-- Hips to Thighs joints -->
-        <xacro:ros2_control_joint joint_name="FLT" lower="-${PI}" upper="${PI}"/>
-        <xacro:ros2_control_joint joint_name="FRT" lower="-${PI}" upper="${PI}"/>
-        <xacro:ros2_control_joint joint_name="BLT" lower="-${PI}" upper="${PI}"/>
-        <xacro:ros2_control_joint joint_name="BRT" lower="-${PI}" upper="${PI}"/>
-        <!-- Thighs to Shanks joints -->
-        <xacro:ros2_control_joint joint_name="FLS" lower="-${5*PI/6}" upper="${5*PI/6}"/>
-        <xacro:ros2_control_joint joint_name="FRS" lower="-${5*PI/6}" upper="${5*PI/6}"/>
-        <xacro:ros2_control_joint joint_name="BLS" lower="-${5*PI/6}" upper="${5*PI/6}"/>
-        <xacro:ros2_control_joint joint_name="BRS" lower="-${5*PI/6}" upper="${5*PI/6}"/>
+        <!-- ROS2 Control core xacro file: -->
+        <xacro:include filename="ros2_control_core.urdf.xacro"/>
     </ros2_control>
     <gazebo>

File: src/meldog_simple_description/description/ros2_control/transmission/transmission_macros.urdf.xacro (robot description, xacro)
@@ -33,13 +33,13 @@
     </xacro:macro>
     <!-- Meldog Transmissions: -->
-    <!-- Trunk to Hips transmissions -->
-    <xacro:SimpleTransmission joint_name="FLH" reduction="9.97" offset="0.0"/>
-    <xacro:SimpleTransmission joint_name="FRH" reduction="9.97" offset="0.0"/>
-    <xacro:SimpleTransmission joint_name="BLH" reduction="9.97" offset="0.0"/>
-    <xacro:SimpleTransmission joint_name="BRH" reduction="9.97" offset="0.0"/>
-    <!-- Thighs to Shanks transmissions -->
-    <xacro:FourBarLinkageTransmission first_joint_name="FLT" second_joint_name="FLS" reduction="9.97" first_offset="0.0" second_offset="0.0"/>
-    <xacro:FourBarLinkageTransmission first_joint_name="FRT" second_joint_name="FRS" reduction="9.97" first_offset="0.0" second_offset="0.0"/>
-    <xacro:FourBarLinkageTransmission first_joint_name="BLT" second_joint_name="BLS" reduction="9.97" first_offset="0.0" second_offset="0.0"/>
-    <xacro:FourBarLinkageTransmission first_joint_name="BRT" second_joint_name="BRS" reduction="9.97" first_offset="0.0" second_offset="0.0"/>
+    <!-- Trunk to Hips transmissions: -->
+    <xacro:SimpleTransmission joint_name="FLH" reduction="${actuator_gear_ratio}" offset="0.0"/>
+    <xacro:SimpleTransmission joint_name="FRH" reduction="${actuator_gear_ratio}" offset="0.0"/>
+    <xacro:SimpleTransmission joint_name="BLH" reduction="${actuator_gear_ratio}" offset="0.0"/>
+    <xacro:SimpleTransmission joint_name="BRH" reduction="${actuator_gear_ratio}" offset="0.0"/>
+    <!-- Thighs to Shanks transmissions: -->
+    <xacro:FourBarLinkageTransmission first_joint_name="FLT" second_joint_name="FLS" reduction="${actuator_gear_ratio}" first_offset="0.0" second_offset="0.0"/>
+    <xacro:FourBarLinkageTransmission first_joint_name="FRT" second_joint_name="FRS" reduction="${actuator_gear_ratio}" first_offset="0.0" second_offset="0.0"/>
+    <xacro:FourBarLinkageTransmission first_joint_name="BLT" second_joint_name="BLS" reduction="${actuator_gear_ratio}" first_offset="0.0" second_offset="0.0"/>
+    <xacro:FourBarLinkageTransmission first_joint_name="BRT" second_joint_name="BRS" reduction="${actuator_gear_ratio}" first_offset="0.0" second_offset="0.0"/>
 </robot>

Commit message: Fixed typo of left feet joint

File: src/meldog_simple_description/description/meldog_core.urdf.xacro (robot description, xacro)
@@ -145,5 +145,5 @@
     </joint>
     <!-- Shank front right to Feet right left -->
-    <joint name="RLF_joint" type="fixed">
+    <joint name="FRF_joint" type="fixed">
         <origin xyz="0.0 0.0 ${-shank_length}" rpy="0.0 0.0 0.0"/>
         <parent link="shank_front_right_link"/>
