Commit message: Successfully launched meldog in custom world in gazebo sim with ros2 control

File: src/meldog_simple_description/description/gazebo/gazebo_macros.urdf.xacro (robot description, xacro)
@@ -4,6 +4,6 @@
     <xacro:property name="kp_value" value="25000.0"/>
     <xacro:property name="kd_value" value="0.15"/>
-    <xacro:property name="mu2_value" value="0.7"/>
-    <xacro:property name="mu2_value" value="0.7"/>
+    <xacro:property name="mu2_value" value="0.9"/>
+    <xacro:property name="mu2_value" value="0.9"/>
     <xacro:property name="maxVel_value" value="0.25"/>
     <xacro:property name="dampingFactor_value" value="0.00"/>

File: src/meldog_simple_description/description/meldog_core.urdf.xacro (robot description, xacro)
@@ -112,5 +112,5 @@
         <child link="shank_front_left_link"/>
         <axis xyz="0.0 -1.0 0.0"/>
-        <xacro:meldog_joint_limits lower ="-${PI/2}" upper = "${PI/2}"/>
+        <xacro:meldog_joint_limits lower ="-${5*PI/6}" upper = "${5*PI/6}"/>
     </joint>
     <!-- Thigh front right to Shank front right -->
@@ -120,5 +120,5 @@
         <child link="shank_front_right_link"/>
         <axis xyz="0.0 -1.0 0.0"/>
-        <xacro:meldog_joint_limits lower ="-${PI/2}" upper = "${PI/2}"/>
+        <xacro:meldog_joint_limits lower ="-${5*PI/6}" upper = "${5*PI/6}"/>
     </joint>
     <!-- Thigh back left to Shank back left -->
@@ -128,5 +128,5 @@
         <child link="shank_back_left_link"/>
         <axis xyz="0.0 1.0 0.0"/>
-        <xacro:meldog_joint_limits lower ="-${PI/2}" upper = "${PI/2}"/>
+        <xacro:meldog_joint_limits lower ="-${5*PI/6}" upper = "${5*PI/6}"/>
     </joint>
     <!-- Thigh back right to Shank back right -->
@@ -136,5 +136,5 @@
         <child link="shank_back_right_link"/>
         <axis xyz="0.0 1.0 0.0"/>
-        <xacro:meldog_joint_limits lower ="-${PI/2}" upper = "${PI/2}"/>
+        <xacro:meldog_joint_limits lower ="-${5*PI/6}" upper = "${5*PI/6}"/>
     </joint>
     <!-- Shank front left to Feet front left -->

File: src/meldog_simple_description/description/ros2_control/ros2_control_gazebo.urdf.xacro (robot description, xacro)
@@ -21,8 +21,8 @@
         <xacro:ros2_control_joint joint_name="BRT" lower="-${PI}" upper="${PI}"/>
         <!-- Thighs to Shanks joints -->
-        <xacro:ros2_control_joint joint_name="FLS" lower="-${PI/2}" upper="${PI/2}"/>
-        <xacro:ros2_control_joint joint_name="FRS" lower="-${PI/2}" upper="${PI/2}"/>
-        <xacro:ros2_control_joint joint_name="BLS" lower="-${PI/2}" upper="${PI/2}"/>
-        <xacro:ros2_control_joint joint_name="BRS" lower="-${PI/2}" upper="${PI/2}"/>
+        <xacro:ros2_control_joint joint_name="FLS" lower="-${5*PI/6}" upper="${5*PI/6}"/>
+        <xacro:ros2_control_joint joint_name="FRS" lower="-${5*PI/6}" upper="${5*PI/6}"/>
+        <xacro:ros2_control_joint joint_name="BLS" lower="-${5*PI/6}" upper="${5*PI/6}"/>
+        <xacro:ros2_control_joint joint_name="BRS" lower="-${5*PI/6}" upper="${5*PI/6}"/>
     </ros2_control>
     <gazebo>
