Commit message: added joint properties

File: src/meldog_simple_twin/urdf/properties.urdf.xacro (robot description, xacro)
@@ -8,3 +8,8 @@
     <xacro:property name="upper_limb_length" value="" />
     <xacro:property name="lower_limb_length_to_foot" value="" />
+    <!-- joint properties -->
+    <xacro:property name="trunk_upper_limb_lower_limit" value="" />
+    <xacro:property name="upper_limb_lower_limb_lower_limit" value="" />
+    <xacro:property name="trunk_upper_limb_upper_limit" value="" />
+    <xacro:property name="upper_limb_lower_limb_upper_limit" value="" />
 </robot>

Commit message: updated joint properties

File: src/meldog_simple_twin/urdf/properties.urdf.xacro (robot description, xacro)
@@ -9,7 +9,15 @@
     <xacro:property name="lower_limb_length_to_foot" value="" />
     <!-- joint properties -->
+        <!-- joint lower movement limits -->
     <xacro:property name="trunk_upper_limb_lower_limit" value="" />
     <xacro:property name="upper_limb_lower_limb_lower_limit" value="" />
+        <!-- joint upper movement limits -->
     <xacro:property name="trunk_upper_limb_upper_limit" value="" />
     <xacro:property name="upper_limb_lower_limb_upper_limit" value="" />
+        <!-- joint effort limits -->
+    <xacro:property name="trunk_upper_limb_effort" value="" />
+    <xacro:property name="upper_limb_lower_limb_effort" value="" />
+        <!-- joint velocity limits -->
+    <xacro:property name="trunk_upper_limb_effort" value="" />
+    <xacro:property name="upper_limb_lower_limb_effort" value="" />
 </robot>

Commit message: implemented properties in urdf, improved readability

File: src/meldog_simple_twin/urdf/properties.urdf.xacro (robot description, xacro)
@@ -1,23 +1,23 @@
 <?xml version="1.0"?>
 <robot xmlns:xacro="http://www.ros.org/wiki/xacro">
-    <!-- stl names for each link in leg -->
+    <!-- stl mesh names for each link in leg -->
     <xacro:property name="trunk_stl_name" value="" />
-    <xacro:property name="upper_limb_stl_name" value="" />
-    <xacro:property name="lower_limb_stl_name" value="" />
+    <xacro:property name="upper_limb_stl_name" value="upper_limb_test.stl" />
+    <xacro:property name="lower_limb_stl_name" value="lower_limb_test.stl" />
     <!-- leg dimensions -->
-    <xacro:property name="upper_limb_length" value="" />
-    <xacro:property name="lower_limb_length_to_foot" value="" />
+    <xacro:property name="upper_limb_length" value="0.25" />
+    <xacro:property name="lower_limb_length_to_foot" value="0.25" />
     <!-- joint properties -->
-        <!-- joint lower movement limits -->
-    <xacro:property name="trunk_upper_limb_lower_limit" value="" />
-    <xacro:property name="upper_limb_lower_limb_lower_limit" value="" />
-        <!-- joint upper movement limits -->
-    <xacro:property name="trunk_upper_limb_upper_limit" value="" />
-    <xacro:property name="upper_limb_lower_limb_upper_limit" value="" />
+        <!-- joint lower movement limits in degrees -->
+    <xacro:property name="trunk_upper_limb_lower_limit" value="0" />
+    <xacro:property name="upper_limb_lower_limb_lower_limit" value="0" />
+        <!-- joint upper movement limits in degrees -->
+    <xacro:property name="trunk_upper_limb_upper_limit" value="90" />
+    <xacro:property name="upper_limb_lower_limb_upper_limit" value="90" />
         <!-- joint effort limits -->
-    <xacro:property name="trunk_upper_limb_effort" value="" />
-    <xacro:property name="upper_limb_lower_limb_effort" value="" />
+    <xacro:property name="trunk_upper_limb_effort" value="100.0" />
+    <xacro:property name="upper_limb_lower_limb_effort" value="100.0" />
         <!-- joint velocity limits -->
-    <xacro:property name="trunk_upper_limb_effort" value="" />
-    <xacro:property name="upper_limb_lower_limb_effort" value="" />
+    <xacro:property name="trunk_upper_limb_velocity" value="100.0" />
+    <xacro:property name="upper_limb_lower_limb_velocity" value="100.0" />
 </robot>

File: src/meldog_simple_twin/urdf/standalone_leg.urdf.xacro (robot description, xacro)
@@ -1,9 +1,10 @@
 <?xml version="1.0"?>
-<robot name="meldog_simple_core" xmlns:xacro="http://www.ros.org/wiki/xacro">
+<robot name="meldog_simple_core"
+    xmlns:xacro="http://www.ros.org/wiki/xacro">
     <xacro:include filename="properties.urdf.xacro" />
     <link name="upper_limb_link">
         <visual>
             <geometry>
-                <mesh filename="package://meldog_simple_twin/meshes/upper_limb_test.stl" scale="0.001 0.001 0.001" />
+                <mesh filename="package://meldog_simple_twin/meshes/${upper_limb_stl_name}" scale="0.001 0.001 0.001" />
             </geometry>
             <origin xyz="0 0 0" rpy="0 0 0"/>
@@ -13,5 +14,5 @@
         <visual>
             <geometry>
-                <mesh filename="package://meldog_simple_twin/meshes/lower_limb_test.stl" scale="0.001 0.001 0.001" />
+                <mesh filename="package://meldog_simple_twin/meshes/${lower_limb_stl_name}" scale="0.001 0.001 0.001" />
             </geometry>
             <origin xyz="0 0 0" rpy="0 0 0"/>
@@ -31,5 +32,8 @@
         <child link="upper_limb_link" />
         <origin xyz="0 0.1 0" rpy="0 0 0" />
-        <limit lower="${-16.0/36.0*2*pi}" upper="${16.0/36.0*2*pi}" effort="100" velocity="100" />
+        <limit lower="${trunk_upper_limb_lower_limit/180.0*pi}"
+               upper="${trunk_upper_limb_upper_limit/180.0*pi}"
+               effort="${trunk_upper_limb_effort}"
+               velocity="${trunk_upper_limb_velocity}" />
         <axis xyz="0 1 0" />
     </joint>
@@ -37,6 +41,9 @@
         <parent link="upper_limb_link" />
         <child link="lower_limb_link" />
-        <origin xyz="0 0 -0.25" rpy="0 0 0" />
-        <limit lower="${-16.0/36.0*2*pi}" upper="${16.0/36.0*2*pi}" effort="100" velocity="100" />
+        <origin xyz="0 0 ${-upper_limb_length}" rpy="0 0 0" />
+        <limit lower="${upper_limb_lower_limb_lower_limit/180.0*pi}"
+               upper="${upper_limb_lower_limb_upper_limit/180.0*pi}"
+               effort="${upper_limb_lower_limb_effort}"
+               velocity="${upper_limb_lower_limb_velocity}" />
         <axis xyz="0 1 0" />
     </joint>
@@ -44,5 +51,5 @@
         <parent link="lower_limb_link" />
         <child link="foot_link" />
-        <origin xyz="0 0 -0.25" rpy="0 0 0" />
+        <origin xyz="0 0 ${-lower_limb_length_to_foot}" rpy="0 0 0" />
     </joint>
 </robot>

Commit message: further improved properties readability

File: src/meldog_simple_twin/urdf/properties.urdf.xacro (robot description, xacro)
@@ -9,15 +9,16 @@
     <xacro:property name="lower_limb_length_to_foot" value="0.25" />
     <!-- joint properties -->
-        <!-- joint lower movement limits in degrees -->
-    <xacro:property name="trunk_upper_limb_lower_limit" value="0" />
-    <xacro:property name="upper_limb_lower_limb_lower_limit" value="0" />
-        <!-- joint upper movement limits in degrees -->
-    <xacro:property name="trunk_upper_limb_upper_limit" value="90" />
-    <xacro:property name="upper_limb_lower_limb_upper_limit" value="90" />
+        <!-- joint movement limits in degrees -->
+            <!-- trunk upper limb joint -->
+            <xacro:property name="trunk_upper_limb_lower_limit" value="0" />
+            <xacro:property name="trunk_upper_limb_upper_limit" value="90" />
+            <!-- upper limb lower limb joint -->
+            <xacro:property name="upper_limb_lower_limb_lower_limit" value="0" />
+            <xacro:property name="upper_limb_lower_limb_upper_limit" value="90" />
         <!-- joint effort limits -->
-    <xacro:property name="trunk_upper_limb_effort" value="100.0" />
-    <xacro:property name="upper_limb_lower_limb_effort" value="100.0" />
+        <xacro:property name="trunk_upper_limb_effort" value="100.0" />
+        <xacro:property name="upper_limb_lower_limb_effort" value="100.0" />
         <!-- joint velocity limits -->
-    <xacro:property name="trunk_upper_limb_velocity" value="100.0" />
-    <xacro:property name="upper_limb_lower_limb_velocity" value="100.0" />
+        <xacro:property name="trunk_upper_limb_velocity" value="100.0" />
+        <xacro:property name="upper_limb_lower_limb_velocity" value="100.0" />
 </robot>

Commit message: renamed leg body link

File: src/meldog_simple_twin/urdf/properties.urdf.xacro (robot description, xacro)
@@ -2,5 +2,5 @@
 <robot xmlns:xacro="http://www.ros.org/wiki/xacro">
     <!-- stl mesh names for each link in leg -->
-    <xacro:property name="trunk_stl_name" value="" />
+    <xacro:property name="leg_body_stl_name" value="" />
     <xacro:property name="upper_limb_stl_name" value="upper_limb_test.stl" />
     <xacro:property name="lower_limb_stl_name" value="lower_limb_test.stl" />
@@ -10,15 +10,15 @@
     <!-- joint properties -->
         <!-- joint movement limits in degrees -->
-            <!-- trunk upper limb joint -->
-            <xacro:property name="trunk_upper_limb_lower_limit" value="0" />
-            <xacro:property name="trunk_upper_limb_upper_limit" value="90" />
+            <!-- leg body upper limb joint -->
+            <xacro:property name="leg_body_upper_limb_lower_limit" value="0" />
+            <xacro:property name="leg_body_upper_limb_upper_limit" value="90" />
             <!-- upper limb lower limb joint -->
             <xacro:property name="upper_limb_lower_limb_lower_limit" value="0" />
             <xacro:property name="upper_limb_lower_limb_upper_limit" value="90" />
         <!-- joint effort limits -->
-        <xacro:property name="trunk_upper_limb_effort" value="100.0" />
+        <xacro:property name="leg_body_upper_limb_effort" value="100.0" />
         <xacro:property name="upper_limb_lower_limb_effort" value="100.0" />
         <!-- joint velocity limits -->
-        <xacro:property name="trunk_upper_limb_velocity" value="100.0" />
+        <xacro:property name="leg_body_upper_limb_velocity" value="100.0" />
         <xacro:property name="upper_limb_lower_limb_velocity" value="100.0" />
 </robot>

File: src/meldog_simple_twin/urdf/standalone_leg.urdf.xacro (robot description, xacro)
@@ -20,5 +20,5 @@
     </link>
     <link name="foot_link" />
-    <link name="trunk_link">
+    <link name="leg_body_link">
         <visual>
             <geometry>
@@ -28,12 +28,12 @@
         </visual>
     </link>
-    <joint name="trunk_upper_limb_joint" type="revolute">
-        <parent link="trunk_link" />
+    <joint name="leg_body_upper_limb_joint" type="revolute">
+        <parent link="leg_body_link" />
         <child link="upper_limb_link" />
         <origin xyz="0 0.1 0" rpy="0 0 0" />
-        <limit lower="${trunk_upper_limb_lower_limit/180.0*pi}"
-               upper="${trunk_upper_limb_upper_limit/180.0*pi}"
-               effort="${trunk_upper_limb_effort}"
-               velocity="${trunk_upper_limb_velocity}" />
+        <limit lower="${leg_body_upper_limb_lower_limit/180.0*pi}"
+               upper="${leg_body_upper_limb_upper_limit/180.0*pi}"
+               effort="${leg_body_upper_limb_effort}"
+               velocity="${leg_body_upper_limb_velocity}" />
         <axis xyz="0 1 0" />
     </joint>
