Commit message: added inertial tags to each link

File: src/meldog_simple_twin/urdf/standalone_leg.urdf.xacro (robot description, xacro)
@@ -18,4 +18,9 @@
             <origin xyz="0 0 0" rpy="0 0 0" />
         </collision>
+        <inertial>
+            <mass value="${}" />
+            <origin xyz="${}" rpy="${}" />
+            <inertia ixx="${}" ixy="${}" ixz="${}" iyy="${}" iyz="${}" izz="${}" />
+        </inertial>
     </link>
     <link name="lower_limb_link">
@@ -34,4 +39,9 @@
             <origin xyz="0 0 0" rpy="0 0 0" />
         </collision>
+        <inertial>
+            <mass value="${}" />
+            <origin xyz="${}" rpy="${}" />
+            <inertia ixx="${}" ixy="${}" ixz="${}" iyy="${}" iyz="${}" izz="${}" />
+        </inertial>
     </link>
     <link name="foot_link" />
@@ -51,4 +61,9 @@
             <origin xyz="0 0 0" rpy="0 0 0" />
         </collision>
+        <inertial>
+            <mass value="${}" />
+            <origin xyz="${}" rpy="${}" />
+            <inertia ixx="${}" ixy="${}" ixz="${}" iyy="${}" iyz="${}" izz="${}" />
+        </inertial>
     </link>
     <joint name="leg_body_upper_limb_joint" type="revolute">
