Commit message: added leg_body_test mesh

File: src/meldog_simple_twin/urdf/base_properties.urdf.xacro (robot description, xacro)
@@ -2,5 +2,5 @@
 <robot xmlns:xacro="http://www.ros.org/wiki/xacro">
     <!-- stl mesh names for each link in leg -->
-    <xacro:property name="leg_body_stl_name" value="" />
+    <xacro:property name="leg_body_stl_name" value="leg_body_test.stl" />
     <xacro:property name="upper_limb_stl_name" value="upper_limb_test.stl" />
     <xacro:property name="lower_limb_stl_name" value="lower_limb_test.stl" />

File: src/meldog_simple_twin/urdf/standalone_leg.urdf.xacro (robot description, xacro)
@@ -23,5 +23,5 @@
         <visual>
             <geometry>
-                <box size="0.3 0.2 0.1" />
+                <mesh filename="package://meldog_simple_twin/meshes/${leg_body_stl_name}" scale="0.001 0.001 0.001" />
             </geometry>
             <origin xyz="0 0 0" rpy="0 0 0" />

Commit message: added leg body joint properties

File: src/meldog_simple_twin/urdf/base_properties.urdf.xacro (robot description, xacro)
@@ -5,14 +5,19 @@
     <xacro:property name="upper_limb_stl_name" value="upper_limb_test.stl" />
     <xacro:property name="lower_limb_stl_name" value="lower_limb_test.stl" />
-    <!-- leg dimensions -->
+    <!-- limb dimensions -->
     <xacro:property name="upper_limb_length" value="0.25" />
     <xacro:property name="lower_limb_length_to_foot" value="0.25" />
     <!-- joint properties -->
+        <!-- body to limb Joint positions -->
+            <!-- leg body upper limb joint -->
+            <xacro:property name="leg_body_upper_limb_x" value="0.174"/>
+            <xacro:property name="leg_body_upper_limb_y" value="0.097"/>
+            <xacro:property name="leg_body_upper_limb_z" value="0"/>
         <!-- joint movement limits in degrees -->
             <!-- leg body upper limb joint -->
-            <xacro:property name="leg_body_upper_limb_lower_limit" value="0" />
+            <xacro:property name="leg_body_upper_limb_lower_limit" value="-90" />
             <xacro:property name="leg_body_upper_limb_upper_limit" value="90" />
             <!-- upper limb lower limb joint -->
-            <xacro:property name="upper_limb_lower_limb_lower_limit" value="0" />
+            <xacro:property name="upper_limb_lower_limb_lower_limit" value="-90" />
             <xacro:property name="upper_limb_lower_limb_upper_limit" value="90" />
         <!-- joint effort limits -->

File: src/meldog_simple_twin/urdf/standalone_leg.urdf.xacro (robot description, xacro)
@@ -31,5 +31,8 @@
         <parent link="leg_body_link" />
         <child link="upper_limb_link" />
-        <origin xyz="0 0.1 0" rpy="0 0 0" />
+        <origin xyz="${leg_body_upper_limb_x}
+                     ${leg_body_upper_limb_y}
+                     ${leg_body_upper_limb_z}"
+                rpy="0 0 0" />
         <limit lower="${leg_body_upper_limb_lower_limit/180.0*pi}"
                upper="${leg_body_upper_limb_upper_limit/180.0*pi}"

Commit message: updated mesh files, corrected joint placement

File: src/meldog_simple_twin/urdf/base_properties.urdf.xacro (robot description, xacro)
@@ -12,5 +12,5 @@
             <!-- leg body upper limb joint -->
             <xacro:property name="leg_body_upper_limb_x" value="0.174"/>
-            <xacro:property name="leg_body_upper_limb_y" value="0.097"/>
+            <xacro:property name="leg_body_upper_limb_y" value="0.0925"/>
             <xacro:property name="leg_body_upper_limb_z" value="0"/>
         <!-- joint movement limits in degrees -->

Commit message: created subfolders for visual and collision meshes, implemented simplified meshes for collision

File: src/meldog_simple_twin/urdf/base_properties.urdf.xacro (robot description, xacro)
@@ -2,7 +2,12 @@
 <robot xmlns:xacro="http://www.ros.org/wiki/xacro">
     <!-- stl mesh names for each link in leg -->
-    <xacro:property name="leg_body_stl_name" value="leg_body_test.stl" />
-    <xacro:property name="upper_limb_stl_name" value="upper_limb_test.stl" />
-    <xacro:property name="lower_limb_stl_name" value="lower_limb_test.stl" />
+        <!-- visual tag meshes -->
+        <xacro:property name="leg_body_vis_stl_name" value="leg_body_test.stl" />
+        <xacro:property name="upper_limb_vis_stl_name" value="upper_limb_test.stl" />
+        <xacro:property name="lower_limb_vis_stl_name" value="lower_limb_test.stl" />
+        <!-- collision tag meshes -->
+        <xacro:property name="leg_body_coll_stl_name" value="leg_body_collision.stl" />
+        <xacro:property name="upper_limb_coll_stl_name" value="upper_limb_collision.stl" />
+        <xacro:property name="lower_limb_coll_stl_name" value="lower_limb_collision.stl" />
     <!-- limb dimensions -->
     <xacro:property name="upper_limb_length" value="0.25" />
@@ -16,9 +21,9 @@
         <!-- joint movement limits in degrees -->
             <!-- leg body upper limb joint -->
-            <xacro:property name="leg_body_upper_limb_lower_limit" value="-90" />
-            <xacro:property name="leg_body_upper_limb_upper_limit" value="90" />
+            <xacro:property name="leg_body_upper_limb_lower_limit" value="-120" />
+            <xacro:property name="leg_body_upper_limb_upper_limit" value="120" />
             <!-- upper limb lower limb joint -->
-            <xacro:property name="upper_limb_lower_limb_lower_limit" value="-90" />
-            <xacro:property name="upper_limb_lower_limb_upper_limit" value="90" />
+            <xacro:property name="upper_limb_lower_limb_lower_limit" value="-160" />
+            <xacro:property name="upper_limb_lower_limb_upper_limit" value="160" />
         <!-- joint effort limits -->
         <xacro:property name="leg_body_upper_limb_effort" value="100.0" />

File: src/meldog_simple_twin/urdf/standalone_leg.urdf.xacro (robot description, xacro)
@@ -6,16 +6,32 @@
         <visual>
             <geometry>
-                <mesh filename="package://meldog_simple_twin/meshes/${upper_limb_stl_name}" scale="0.001 0.001 0.001" />
+                <mesh filename="package://meldog_simple_twin/meshes/visual/${upper_limb_vis_stl_name}"
+                      scale="0.001 0.001 0.001" />
             </geometry>
             <origin xyz="0 0 0" rpy="0 0 0"/>
         </visual>
+        <collision>
+            <geometry>
+                <mesh filename="package://meldog_simple_twin/meshes/collision/${upper_limb_coll_stl_name}"
+                      scale="0.001 0.001 0.001" />
+            </geometry>
+            <origin xyz="0 0 0" rpy="0 0 0" />
+        </collision>
     </link>
     <link name="lower_limb_link">
         <visual>
             <geometry>
-                <mesh filename="package://meldog_simple_twin/meshes/${lower_limb_stl_name}" scale="0.001 0.001 0.001" />
+                <mesh filename="package://meldog_simple_twin/meshes/visual/${lower_limb_vis_stl_name}"
+                      scale="0.001 0.001 0.001" />
             </geometry>
             <origin xyz="0 0 0" rpy="0 0 0"/>
         </visual>
+        <collision>
+            <geometry>
+                <mesh filename="package://meldog_simple_twin/meshes/collision/${lower_limb_coll_stl_name}"
+                      scale="0.001 0.001 0.001" />
+            </geometry>
+            <origin xyz="0 0 0" rpy="0 0 0" />
+        </collision>
     </link>
     <link name="foot_link" />
@@ -23,8 +39,16 @@
         <visual>
             <geometry>
-                <mesh filename="package://meldog_simple_twin/meshes/${leg_body_stl_name}" scale="0.001 0.001 0.001" />
+                <mesh filename="package://meldog_simple_twin/meshes/visual/${leg_body_vis_stl_name}"
+                      scale="0.001 0.001 0.001" />
             </geometry>
             <origin xyz="0 0 0" rpy="0 0 0" />
         </visual>
+        <collision>
+            <geometry>
+                <mesh filename="package://meldog_simple_twin/meshes/collision/${leg_body_coll_stl_name}"
+                      scale="0.001 0.001 0.001" />
+            </geometry>
+            <origin xyz="0 0 0" rpy="0 0 0" />
+        </collision>
     </link>
     <joint name="leg_body_upper_limb_joint" type="revolute">

Commit message: declared inertial properties for each link in properties file

File: src/meldog_simple_twin/urdf/base_properties.urdf.xacro (robot description, xacro)
@@ -13,4 +13,47 @@
     <xacro:property name="upper_limb_length" value="0.25" />
     <xacro:property name="lower_limb_length_to_foot" value="0.25" />
+    <!-- inertial properties for each link -->
+        <!-- leg body link -->
+            <!-- mass -->
+            <xacro:property name="leg_body_mass" value=""/>
+            <!-- center of mass -->
+            <xacro:property name="leg_body_cm_x" value=""/>
+            <xacro:property name="leg_body_cm_y" value=""/>
+            <xacro:property name="leg_body_cm_z" value=""/>
+            <!-- moments of inertia -->
+            <xacro:property name="leg_body_ixx" value=""/>
+            <xacro:property name="leg_body_ixy" value=""/>
+            <xacro:property name="leg_body_ixz" value=""/>
+            <xacro:property name="leg_body_iyy" value=""/>
+            <xacro:property name="leg_body_iyz" value=""/>
+            <xacro:property name="leg_body_izz" value=""/>
+        <!-- upper limb link -->
+            <!-- mass -->
+            <xacro:property name="leg_body_mass" value=""/>
+            <!-- center of mass -->
+            <xacro:property name="leg_body_cm_x" value=""/>
+            <xacro:property name="leg_body_cm_y" value=""/>
+            <xacro:property name="leg_body_cm_z" value=""/>
+            <!-- moments of inertia -->
+            <xacro:property name="leg_body_ixx" value=""/>
+            <xacro:property name="leg_body_ixy" value=""/>
+            <xacro:property name="leg_body_ixz" value=""/>
+            <xacro:property name="leg_body_iyy" value=""/>
+            <xacro:property name="leg_body_iyz" value=""/>
+            <xacro:property name="leg_body_izz" value=""/>
+        <!-- lower limb link -->
+            <!-- mass -->
+            <xacro:property name="leg_body_mass" value=""/>
+            <!-- center of mass -->
+            <xacro:property name="leg_body_cm_x" value=""/>
+            <xacro:property name="leg_body_cm_y" value=""/>
+            <xacro:property name="leg_body_cm_z" value=""/>
+            <!-- moments of inertia -->
+            <xacro:property name="leg_body_ixx" value=""/>
+            <xacro:property name="leg_body_ixy" value=""/>
+            <xacro:property name="leg_body_ixz" value=""/>
+            <xacro:property name="leg_body_iyy" value=""/>
+            <xacro:property name="leg_body_iyz" value=""/>
+            <xacro:property name="leg_body_izz" value=""/>
     <!-- joint properties -->
         <!-- body to limb Joint positions -->

Commit message: filled inertia tags with xacro parameters

File: src/meldog_simple_twin/urdf/base_properties.urdf.xacro (robot description, xacro)
@@ -16,44 +16,44 @@
         <!-- leg body link -->
             <!-- mass -->
-            <xacro:property name="leg_body_mass" value=""/>
+            <xacro:property name="leg_body_mass" value="0"/>
             <!-- center of mass -->
-            <xacro:property name="leg_body_cm_x" value=""/>
-            <xacro:property name="leg_body_cm_y" value=""/>
-            <xacro:property name="leg_body_cm_z" value=""/>
+            <xacro:property name="leg_body_cm_x" value="0"/>
+            <xacro:property name="leg_body_cm_y" value="0"/>
+            <xacro:property name="leg_body_cm_z" value="0"/>
             <!-- moments of inertia -->
-            <xacro:property name="leg_body_ixx" value=""/>
-            <xacro:property name="leg_body_ixy" value=""/>
-            <xacro:property name="leg_body_ixz" value=""/>
-            <xacro:property name="leg_body_iyy" value=""/>
-            <xacro:property name="leg_body_iyz" value=""/>
-            <xacro:property name="leg_body_izz" value=""/>
+            <xacro:property name="leg_body_ixx" value="0"/>
+            <xacro:property name="leg_body_ixy" value="0"/>
+            <xacro:property name="leg_body_ixz" value="0"/>
+            <xacro:property name="leg_body_iyy" value="0"/>
+            <xacro:property name="leg_body_iyz" value="0"/>
+            <xacro:property name="leg_body_izz" value="0"/>
         <!-- upper limb link -->
             <!-- mass -->
-            <xacro:property name="leg_body_mass" value=""/>
+            <xacro:property name="upper_limb_mass" value="0"/>
             <!-- center of mass -->
-            <xacro:property name="leg_body_cm_x" value=""/>
-            <xacro:property name="leg_body_cm_y" value=""/>
-            <xacro:property name="leg_body_cm_z" value=""/>
+            <xacro:property name="upper_limb_cm_x" value="0"/>
+            <xacro:property name="upper_limb_cm_y" value="0"/>
+            <xacro:property name="upper_limb_cm_z" value="0"/>
             <!-- moments of inertia -->
-            <xacro:property name="leg_body_ixx" value=""/>
-            <xacro:property name="leg_body_ixy" value=""/>
-            <xacro:property name="leg_body_ixz" value=""/>
-            <xacro:property name="leg_body_iyy" value=""/>
-            <xacro:property name="leg_body_iyz" value=""/>
-            <xacro:property name="leg_body_izz" value=""/>
+            <xacro:property name="upper_limb_ixx" value="0"/>
+            <xacro:property name="upper_limb_ixy" value="0"/>
+            <xacro:property name="upper_limb_ixz" value="0"/>
+            <xacro:property name="upper_limb_iyy" value="0"/>
+            <xacro:property name="upper_limb_iyz" value="0"/>
+            <xacro:property name="upper_limb_izz" value="0"/>
         <!-- lower limb link -->
             <!-- mass -->
-            <xacro:property name="leg_body_mass" value=""/>
+            <xacro:property name="lower_limb_mass" value="0"/>
             <!-- center of mass -->
-            <xacro:property name="leg_body_cm_x" value=""/>
-            <xacro:property name="leg_body_cm_y" value=""/>
-            <xacro:property name="leg_body_cm_z" value=""/>
+            <xacro:property name="lower_limb_cm_x" value="0"/>
+            <xacro:property name="lower_limb_cm_y" value="0"/>
+            <xacro:property name="lower_limb_cm_z" value="0"/>
             <!-- moments of inertia -->
-            <xacro:property name="leg_body_ixx" value=""/>
-            <xacro:property name="leg_body_ixy" value=""/>
-            <xacro:property name="leg_body_ixz" value=""/>
-            <xacro:property name="leg_body_iyy" value=""/>
-            <xacro:property name="leg_body_iyz" value=""/>
-            <xacro:property name="leg_body_izz" value=""/>
+            <xacro:property name="lower_limb_ixx" value="0"/>
+            <xacro:property name="lower_limb_ixy" value="0"/>
+            <xacro:property name="lower_limb_ixz" value="0"/>
+            <xacro:property name="lower_limb_iyy" value="0"/>
+            <xacro:property name="lower_limb_iyz" value="0"/>
+            <xacro:property name="lower_limb_izz" value="0"/>
     <!-- joint properties -->
         <!-- body to limb Joint positions -->

File: src/meldog_simple_twin/urdf/standalone_leg.urdf.xacro (robot description, xacro)
@@ -19,7 +19,9 @@
         </collision>
         <inertial>
-            <mass value="${}" />
-            <origin xyz="${}" rpy="${}" />
-            <inertia ixx="${}" ixy="${}" ixz="${}" iyy="${}" iyz="${}" izz="${}" />
+            <mass value="${upper_limb_mass}" />
+            <origin xyz="${upper_limb_cm_x} ${upper_limb_cm_y} ${upper_limb_cm_z}" rpy="0 0 0" />
+            <inertia ixx="${upper_limb_ixx}" ixy="${upper_limb_ixy}" ixz="${upper_limb_ixz}"
+                                             iyy="${upper_limb_iyy}" iyz="${upper_limb_iyz}"
+                                                                     izz="${upper_limb_izz}" />
         </inertial>
     </link>
@@ -40,7 +42,9 @@
         </collision>
         <inertial>
-            <mass value="${}" />
-            <origin xyz="${}" rpy="${}" />
-            <inertia ixx="${}" ixy="${}" ixz="${}" iyy="${}" iyz="${}" izz="${}" />
+            <mass value="${lower_limb_mass}" />
+            <origin xyz="${lower_limb_cm_x} ${lower_limb_cm_y} ${lower_limb_cm_z}" rpy="0 0 0" />
+            <inertia ixx="${lower_limb_ixx}" ixy="${lower_limb_ixy}" ixz="${lower_limb_ixz}"
+                                             iyy="${lower_limb_iyy}" iyz="${lower_limb_iyz}"
+                                                                     izz="${lower_limb_izz}" />
         </inertial>
     </link>
@@ -62,7 +66,9 @@
         </collision>
         <inertial>
-            <mass value="${}" />
-            <origin xyz="${}" rpy="${}" />
-            <inertia ixx="${}" ixy="${}" ixz="${}" iyy="${}" iyz="${}" izz="${}" />
+            <mass value="${leg_body_mass}" />
+            <origin xyz="${leg_body_cm_x} ${leg_body_cm_y} ${leg_body_cm_z}" rpy="0 0 0" />
+            <inertia ixx="${leg_body_ixx}" ixy="${leg_body_ixy}" ixz="${leg_body_ixz}"
+                                           iyy="${leg_body_iyy}" iyz="${leg_body_iyz}"
+                                                                 izz="${leg_body_izz}" />
         </inertial>
     </link>

Commit message: inserted calculeted inertial properties of links

File: src/meldog_simple_twin/urdf/base_properties.urdf.xacro (robot description, xacro)
@@ -16,44 +16,44 @@
         <!-- leg body link -->
             <!-- mass -->
-            <xacro:property name="leg_body_mass" value="0"/>
+            <xacro:property name="leg_body_mass" value="3.607"/>
             <!-- center of mass -->
-            <xacro:property name="leg_body_cm_x" value="0"/>
-            <xacro:property name="leg_body_cm_y" value="0"/>
-            <xacro:property name="leg_body_cm_z" value="0"/>
+            <xacro:property name="leg_body_cm_x" value="125.497"/>
+            <xacro:property name="leg_body_cm_y" value="20.770"/>
+            <xacro:property name="leg_body_cm_z" value="0.248"/>
             <!-- moments of inertia -->
-            <xacro:property name="leg_body_ixx" value="0"/>
-            <xacro:property name="leg_body_ixy" value="0"/>
-            <xacro:property name="leg_body_ixz" value="0"/>
-            <xacro:property name="leg_body_iyy" value="0"/>
-            <xacro:property name="leg_body_iyz" value="0"/>
-            <xacro:property name="leg_body_izz" value="0"/>
+            <xacro:property name="leg_body_ixx" value="4660.408"/>
+            <xacro:property name="leg_body_ixy" value="-338.226"/>
+            <xacro:property name="leg_body_ixz" value="0.847"/>
+            <xacro:property name="leg_body_iyy" value="14607.423"/>
+            <xacro:property name="leg_body_iyz" value="49.927"/>
+            <xacro:property name="leg_body_izz" value="13707.172"/>
         <!-- upper limb link -->
             <!-- mass -->
-            <xacro:property name="upper_limb_mass" value="0"/>
+            <xacro:property name="upper_limb_mass" value="0.474"/>
             <!-- center of mass -->
-            <xacro:property name="upper_limb_cm_x" value="0"/>
-            <xacro:property name="upper_limb_cm_y" value="0"/>
-            <xacro:property name="upper_limb_cm_z" value="0"/>
+            <xacro:property name="upper_limb_cm_x" value="-1.185"/>
+            <xacro:property name="upper_limb_cm_y" value="-4.308"/>
+            <xacro:property name="upper_limb_cm_z" value="-94.203"/>
             <!-- moments of inertia -->
-            <xacro:property name="upper_limb_ixx" value="0"/>
-            <xacro:property name="upper_limb_ixy" value="0"/>
-            <xacro:property name="upper_limb_ixz" value="0"/>
-            <xacro:property name="upper_limb_iyy" value="0"/>
-            <xacro:property name="upper_limb_iyz" value="0"/>
-            <xacro:property name="upper_limb_izz" value="0"/>
+            <xacro:property name="upper_limb_ixx" value="4064.505"/>
+            <xacro:property name="upper_limb_ixy" value="1.241"/>
+            <xacro:property name="upper_limb_ixz" value="19.989"/>
+            <xacro:property name="upper_limb_iyy" value="4150.05"/>
+            <xacro:property name="upper_limb_iyz" value="235.648"/>
+            <xacro:property name="upper_limb_izz" value="424.555"/>
         <!-- lower limb link -->
             <!-- mass -->
-            <xacro:property name="lower_limb_mass" value="0"/>
+            <xacro:property name="lower_limb_mass" value="0.116"/>
             <!-- center of mass -->
-            <xacro:property name="lower_limb_cm_x" value="0"/>
+            <xacro:property name="lower_limb_cm_x" value="0.546"/>
             <xacro:property name="lower_limb_cm_y" value="0"/>
-            <xacro:property name="lower_limb_cm_z" value="0"/>
+            <xacro:property name="lower_limb_cm_z" value="-177.643"/>
             <!-- moments of inertia -->
-            <xacro:property name="lower_limb_ixx" value="0"/>
+            <xacro:property name="lower_limb_ixx" value="967.349"/>
             <xacro:property name="lower_limb_ixy" value="0"/>
-            <xacro:property name="lower_limb_ixz" value="0"/>
-            <xacro:property name="lower_limb_iyy" value="0"/>
-            <xacro:property name="lower_limb_iyz" value="0"/>
-            <xacro:property name="lower_limb_izz" value="0"/>
+            <xacro:property name="lower_limb_ixz" value="-4.842"/>
+            <xacro:property name="lower_limb_iyy" value="982.604"/>
+            <xacro:property name="lower_limb_iyz" value="-0.001"/>
+            <xacro:property name="lower_limb_izz" value="37.177"/>
     <!-- joint properties -->
         <!-- body to limb Joint positions -->
