Commit message: added link subdivision folders and macros file

File: src/meldog_description/description/standalone_leg.urdf.xacro (robot description, xacro)
@@ -50,5 +50,5 @@
     </link>
     <link name="foot_link" />
-    <link name="leg_body_link">
+    <link name="hip_link">
         <visual>
             <geometry>
@@ -73,6 +73,6 @@
         </inertial>
     </link>
-    <joint name="leg_body_upper_limb_joint" type="revolute">
-        <parent link="leg_body_link" />
+    <joint name="hip_upper_limb_joint" type="revolute">
+        <parent link="hip_link" />
         <child link="upper_limb_link" />
         <origin xyz="${leg_body_upper_limb_x}
