Commit message: implemented link macros for each link, changed leg_body properties to hip properties

File: src/meldog_description/description/base_properties.urdf.xacro (robot description, xacro)
@@ -3,9 +3,9 @@
     <!-- stl mesh names for each link in leg -->
         <!-- visual tag meshes -->
-        <xacro:property name="leg_body_vis_stl_name" value="leg_body_test.stl" />
+        <xacro:property name="hip_vis_stl_name" value="hip_test.stl" />
         <xacro:property name="upper_limb_vis_stl_name" value="upper_limb_test.stl" />
         <xacro:property name="lower_limb_vis_stl_name" value="lower_limb_test.stl" />
         <!-- collision tag meshes -->
-        <xacro:property name="leg_body_coll_stl_name" value="leg_body_collision.stl" />
+        <xacro:property name="hip_coll_stl_name" value="hip_collision.stl" />
         <xacro:property name="upper_limb_coll_stl_name" value="upper_limb_collision.stl" />
         <xacro:property name="lower_limb_coll_stl_name" value="lower_limb_collision.stl" />
@@ -16,16 +16,16 @@
         <!-- leg body link -->
             <!-- mass -->
-            <xacro:property name="leg_body_mass" value="3.607"/>
+            <xacro:property name="hip_mass" value="3.607"/>
             <!-- center of mass -->
-            <xacro:property name="leg_body_cm_x" value="125.497"/>
-            <xacro:property name="leg_body_cm_y" value="20.770"/>
-            <xacro:property name="leg_body_cm_z" value="0.248"/>
+            <xacro:property name="hip_cm_x" value="125.497"/>
+            <xacro:property name="hip_cm_y" value="20.770"/>
+            <xacro:property name="hip_cm_z" value="0.248"/>
             <!-- moments of inertia -->
-            <xacro:property name="leg_body_ixx" value="4660.408"/>
-            <xacro:property name="leg_body_ixy" value="-338.226"/>
-            <xacro:property name="leg_body_ixz" value="0.847"/>
-            <xacro:property name="leg_body_iyy" value="14607.423"/>
-            <xacro:property name="leg_body_iyz" value="49.927"/>
-            <xacro:property name="leg_body_izz" value="13707.172"/>
+            <xacro:property name="hip_ixx" value="4660.408"/>
+            <xacro:property name="hip_ixy" value="-338.226"/>
+            <xacro:property name="hip_ixz" value="0.847"/>
+            <xacro:property name="hip_iyy" value="14607.423"/>
+            <xacro:property name="hip_iyz" value="49.927"/>
+            <xacro:property name="hip_izz" value="13707.172"/>
         <!-- upper limb link -->
             <!-- mass -->
@@ -59,19 +59,19 @@
         <!-- body to limb Joint positions -->
             <!-- leg body upper limb joint -->
-            <xacro:property name="leg_body_upper_limb_x" value="0.174"/>
-            <xacro:property name="leg_body_upper_limb_y" value="0.0925"/>
-            <xacro:property name="leg_body_upper_limb_z" value="0"/>
+            <xacro:property name="hip_upper_limb_x" value="0.174"/>
+            <xacro:property name="hip_upper_limb_y" value="0.0925"/>
+            <xacro:property name="hip_upper_limb_z" value="0"/>
         <!-- joint movement limits in degrees -->
             <!-- leg body upper limb joint -->
-            <xacro:property name="leg_body_upper_limb_lower_limit" value="-120" />
-            <xacro:property name="leg_body_upper_limb_upper_limit" value="120" />
+            <xacro:property name="hip_upper_limb_lower_limit" value="-120" />
+            <xacro:property name="hip_upper_limb_upper_limit" value="120" />
             <!-- upper limb lower limb joint -->
             <xacro:property name="upper_limb_lower_limb_lower_limit" value="-160" />
             <xacro:property name="upper_limb_lower_limb_upper_limit" value="160" />
         <!-- joint effort limits -->
-        <xacro:property name="leg_body_upper_limb_effort" value="100.0" />
+        <xacro:property name="hip_upper_limb_effort" value="100.0" />
         <xacro:property name="upper_limb_lower_limb_effort" value="100.0" />
         <!-- joint velocity limits -->
-        <xacro:property name="leg_body_upper_limb_velocity" value="100.0" />
+        <xacro:property name="hip_upper_limb_velocity" value="100.0" />
         <xacro:property name="upper_limb_lower_limb_velocity" value="100.0" />
 </robot>

File: src/meldog_description/description/macros/macros.urdf.xacro (robot description, xacro)
@@ -1,6 +1,9 @@
 <?xml version="1.0"?>
 <robot xmlns:xacro="http://www.ros.org/wiki/xacro">
-    <xacro:macro name="link_macro" params="prefix vis_name coll_name m cm_x cm_y cm_z ixx ixy ixz iyy iyz izz">
-        <link name="${prefix}_link">
+    <!-- Macro for defining a link, please ensure that
+    the visual and collision models coordinate
+    systems are placed in joints -->
+    <xacro:macro name="link_macro" params="name vis_name coll_name m cm_x cm_y cm_z ixx ixy ixz iyy iyz izz">
+        <link name="${name}">
             <visual>
                 <geometry>

File: src/meldog_description/description/standalone_leg.urdf.xacro (robot description, xacro)
@@ -2,85 +2,50 @@
 <robot name="meldog_simple_core" xmlns:xacro="http://www.ros.org/wiki/xacro">
     <xacro:include filename="base_properties.urdf.xacro" />
-    <link name="upper_limb_link">
-        <visual>
-            <geometry>
-                <mesh filename="package://meldog_description/meshes/visual/${upper_limb_vis_stl_name}"
-                      scale="0.001 0.001 0.001" />
-            </geometry>
-            <origin xyz="0 0 0" rpy="0 0 0"/>
-        </visual>
-        <collision>
-            <geometry>
-                <mesh filename="package://meldog_description/meshes/collision/${upper_limb_coll_stl_name}"
-                      scale="0.001 0.001 0.001" />
-            </geometry>
-            <origin xyz="0 0 0" rpy="0 0 0" />
-        </collision>
-        <inertial>
-            <mass value="${upper_limb_mass}" />
-            <origin xyz="${upper_limb_cm_x*0.001} ${upper_limb_cm_y*0.001} ${upper_limb_cm_z*0.001}" rpy="0 0 0" />
-            <inertia ixx="${upper_limb_ixx*0.000001}" ixy="${upper_limb_ixy*0.000001}" ixz="${upper_limb_ixz*0.000001}"
-                                                      iyy="${upper_limb_iyy*0.000001}" iyz="${upper_limb_iyz*0.000001}"
-                                                                                       izz="${upper_limb_izz*0.000001}" />
-        </inertial>
-    </link>
-    <link name="lower_limb_link">
-        <visual>
-            <geometry>
-                <mesh filename="package://meldog_description/meshes/visual/${lower_limb_vis_stl_name}"
-                      scale="0.001 0.001 0.001" />
-            </geometry>
-            <origin xyz="0 0 0" rpy="0 0 0"/>
-        </visual>
-        <collision>
-            <geometry>
-                <mesh filename="package://meldog_description/meshes/collision/${lower_limb_coll_stl_name}"
-                      scale="0.001 0.001 0.001" />
-            </geometry>
-            <origin xyz="0 0 0" rpy="0 0 0" />
-        </collision>
-        <inertial>
-            <mass value="${lower_limb_mass}" />
-            <origin xyz="${lower_limb_cm_x*0.001} ${lower_limb_cm_y*0.001} ${lower_limb_cm_z*0.001}" rpy="0 0 0" />
-            <inertia ixx="${lower_limb_ixx*0.000001}" ixy="${lower_limb_ixy*0.000001}" ixz="${lower_limb_ixz*0.000001}"
-                                                      iyy="${lower_limb_iyy*0.000001}" iyz="${lower_limb_iyz*0.000001}"
-                                                                                       izz="${lower_limb_izz*0.000001}" />
-        </inertial>
-    </link>
+    <xacro:include filename="macros/macros.urdf.xacro" />
+    <xacro:link_macro
+        name="upper_limb_link"
+        vis_name="${upper_limb_vis_stl_name}"
+        coll_name="${upper_limb_coll_stl_name}"
+        m="${upper_limb_mass}"
+        cm_x="${upper_limb_cm_x}"
+        cm_y="${upper_limb_cm_y}"
+        cm_z="${upper_limb_cm_z}"
+        ixx="${upper_limb_ixx}" ixy="${upper_limb_ixy}" ixz="${upper_limb_ixz}"
+                                iyy="${upper_limb_iyy}" iyz="${upper_limb_iyz}"
+                                                        izz="${upper_limb_izz}"/>
+    <xacro:link_macro
+        name="lower_limb_link"
+        vis_name="${lower_limb_vis_stl_name}"
+        coll_name="${lower_limb_coll_stl_name}"
+        m="${lower_limb_mass}"
+        cm_x="${lower_limb_cm_x}"
+        cm_y="${lower_limb_cm_y}"
+        cm_z="${lower_limb_cm_z}"
+        ixx="${lower_limb_ixx}" ixy="${lower_limb_ixy}" ixz="${lower_limb_ixz}"
+                                iyy="${lower_limb_iyy}" iyz="${lower_limb_iyz}"
+                                                        izz="${lower_limb_izz}"/>
     <link name="foot_link" />
-    <link name="hip_link">
-        <visual>
-            <geometry>
-                <mesh filename="package://meldog_description/meshes/visual/${leg_body_vis_stl_name}"
-                      scale="0.001 0.001 0.001" />
-            </geometry>
-            <origin xyz="0 0 0" rpy="0 0 0" />
-        </visual>
-        <collision>
-            <geometry>
-                <mesh filename="package://meldog_description/meshes/collision/${leg_body_coll_stl_name}"
-                      scale="0.001 0.001 0.001" />
-            </geometry>
-            <origin xyz="0 0 0" rpy="0 0 0" />
-        </collision>
-        <inertial>
-            <mass value="${leg_body_mass}" />
-            <origin xyz="${leg_body_cm_x*0.001} ${leg_body_cm_y*0.001} ${leg_body_cm_z*0.001}" rpy="0 0 0" />
-            <inertia ixx="${leg_body_ixx*0.000001}" ixy="${leg_body_ixy*0.000001}" ixz="${leg_body_ixz*0.000001}"
-                                                    iyy="${leg_body_iyy*0.000001}" iyz="${leg_body_iyz*0.000001}"
-                                                                                   izz="${leg_body_izz*0.000001}" />
-        </inertial>
-    </link>
+    <xacro:link_macro
+        name="hip_link"
+        vis_name="${hip_vis_stl_name}"
+        coll_name="${hip_coll_stl_name}"
+        m="${hip_mass}"
+        cm_x="${hip_cm_x}"
+        cm_y="${hip_cm_y}"
+        cm_z="${hip_cm_z}"
+        ixx="${hip_ixx}" ixy="${hip_ixy}" ixz="${hip_ixz}"
+                         iyy="${hip_iyy}" iyz="${hip_iyz}"
+                                          izz="${hip_izz}"/>
     <joint name="hip_upper_limb_joint" type="revolute">
         <parent link="hip_link" />
         <child link="upper_limb_link" />
-        <origin xyz="${leg_body_upper_limb_x}
-                     ${leg_body_upper_limb_y}
-                     ${leg_body_upper_limb_z}"
+        <origin xyz="${hip_upper_limb_x}
+                     ${hip_upper_limb_y}
+                     ${hip_upper_limb_z}"
                 rpy="0 0 0" />
-        <limit lower="${leg_body_upper_limb_lower_limit/180.0*pi}"
-               upper="${leg_body_upper_limb_upper_limit/180.0*pi}"
-               effort="${leg_body_upper_limb_effort}"
-               velocity="${leg_body_upper_limb_velocity}" />
+        <limit lower="${hip_upper_limb_lower_limit/180.0*pi}"
+               upper="${hip_upper_limb_upper_limit/180.0*pi}"
+               effort="${hip_upper_limb_effort}"
+               velocity="${hip_upper_limb_velocity}" />
         <axis xyz="0 1 0" />
     </joint>

Commit message: added trunk link from meldog_simple_description package, renamed main urdf file

File: src/meldog_description/description/base_properties.urdf.xacro (robot description, xacro)
@@ -69,9 +69,14 @@
             <xacro:property name="upper_limb_lower_limb_lower_limit" value="-160" />
             <xacro:property name="upper_limb_lower_limb_upper_limit" value="160" />
+            <!-- trunk hip joint -->
+            <xacro:property name="trunk_hip_lower_limit" value="-45" />
+            <xacro:property name="trunk_hip_upper_limit" value="45" />
         <!-- joint effort limits -->
         <xacro:property name="hip_upper_limb_effort" value="100.0" />
         <xacro:property name="upper_limb_lower_limb_effort" value="100.0" />
+        <xacro:property name="trunk_hip_effort" value="100.0" />
         <!-- joint velocity limits -->
         <xacro:property name="hip_upper_limb_velocity" value="100.0" />
         <xacro:property name="upper_limb_lower_limb_velocity" value="100.0" />
+        <xacro:property name="trunk_hip_velocity" value="100.0" />
 </robot>

File: src/meldog_description/description/meldog_core.urdf.xacro (robot description, xacro)
@@ -3,4 +3,5 @@
     <xacro:include filename="base_properties.urdf.xacro" />
     <xacro:include filename="macros/macros.urdf.xacro" />
+    <xacro:include filename="trunk.urdf.xacro" />
     <xacro:link_macro
         name="upper_limb_link"
@@ -65,3 +66,13 @@
         <origin xyz="0 0 ${-lower_limb_length_to_foot}" rpy="0 0 0" />
     </joint>
+    <joint name="trunk_hip_joint" type="revolute">
+        <parent link="trunk_link" />
+        <child link="hip_link" />
+        <origin xyz="${trunk_actuators_length/2.0} ${(trunk_base_width+trunk_actuators_width)/2.0} 0" rpy="0 0 0" />
+        <limit lower="${trunk_hip_lower_limit/180.0*pi}"
+               upper="${trunk_hip_upper_limit/180.0*pi}"
+               effort="${trunk_hip_effort}"
+               velocity="${trunk_hip_velocity}" />
+        <axis xyz="1 0 0" />
+    </joint>
 </robot>

File: src/meldog_description/description/trunk.urdf.xacro (robot description, xacro)
@@ -6,5 +6,5 @@
     <xacro:property name="trunk_base_height" value="0.1" />
     <xacro:property name="trunk_actuators_length" value="0.3" />
-    <xacro:property name="trunk_actuators_width" value="0.1" />
+    <xacro:property name="trunk_actuators_width" value="0.15" />
     <xacro:property name="trunk_actuators_height" value="0.1" />
     <xacro:property name="trunk_mass" value="8.0"/>
