Commit message: Hip links and joints added

File: src/meldog_description/description/meldog_core.urdf.xacro (robot description, xacro)
@@ -1,6 +1,54 @@
 <?xml version="1.0"?>
 <robot xmlns:xacro="http://www.ros.org/wiki/xacro" name = "meldog_core">
-    <!-- BASE LINK spawns in x= 0.0 y = 0.0 z = 0.0-->
+    <!-- PI -->
+    <xacro:property name="PI" value="3.1415926535897"/>
+    <!-- Base link spawns in x= 0.0 y = 0.0 z = 0.0 -->
     <link name="base_link"></link>
+    <!-- Trunk link -->
     <xacro:include filename="trunk/trunk.urdf.xacro"/>
+    <!-- Hip links -->
+    <xacro:include filename="hip/hip.urdf.xacro"/>
+    <xacro:hip_link position="front_left"/>
+    <xacro:hip_link position="front_right"/>
+    <xacro:hip_link position="back_left"/>
+    <xacro:hip_link position="back_right"/>
+    <!-- Base to Trunk joint -->
+    <joint name="base_trunk_joint" type="fixed">
+        <parent link="base_link"/>
+        <child link="trunk_link"/>
+        <!--Origin defines translation child frame relative to parent frame. Translation is performed in parent frame.-->
+        <origin xyz="0 0 1.0" rpy="0 0 0"/>  <!--testing-->
+    </joint>
+    <!-- Trunk to Hip front left joint -->
+    <joint name="trunk_hip_front_left_joint" type="revolute">
+        <origin xyz="${trunk_actuators_length/2} ${trunk_base_width/2 + trunk_actuators_width/2} 0.0" rpy="0.0 0.0 0.0"/>
+        <parent link="trunk_link"/>
+        <child link="hip_front_left_link"/>
+        <axis xyz="1.0 0.0 0.0"/>
+        <limit lower="-1.0" upper="1" effort="10.0" velocity="100.0"/>
+    </joint>
+    <!-- Trunk to Hip front right joint -->
+    <joint name="trunk_hip_front_right_joint" type="revolute">
+        <origin xyz="${trunk_actuators_length/2} ${-(trunk_base_width/2 + trunk_actuators_width/2)} 0.0" rpy="0.0 0.0 0.0"/>
+        <parent link="trunk_link"/>
+        <child link="hip_front_right_link"/>
+        <axis xyz="1.0 0.0 0.0"/>
+        <limit lower="-1.0" upper="1" effort="10.0" velocity="100.0"/>
+    </joint>
+    <!-- Trunk to Hip back left joint -->
+    <joint name="trunk_hip_back_left_joint" type="revolute">
+        <origin xyz="${-trunk_actuators_length/2} ${trunk_base_width/2 + trunk_actuators_width/2} 0.0" rpy="0.0 0.0 ${PI}"/>
+        <parent link="trunk_link"/>
+        <child link="hip_back_left_link"/>
+        <axis xyz="1.0 0.0 0.0"/>
+        <limit lower="-1.0" upper="1" effort="10.0" velocity="100.0"/>
+    </joint>
+    <!-- Trunk to Hip back right joint -->
+    <joint name="trunk_hip_back_right_joint" type="revolute">
+        <origin xyz="${-trunk_actuators_length/2} ${-(trunk_base_width/2 + trunk_actuators_width/2)} 0.0" rpy="0.0 0.0 ${PI}"/>
+        <parent link="trunk_link"/>
+        <child link="hip_back_right_link"/>
+        <axis xyz="1.0 0.0 0.0"/>
+        <limit lower="-1.0" upper="1" effort="10.0" velocity="100.0"/>
+    </joint>
 </robot>

File: src/meldog_description/description/trunk/trunk.urdf.xacro (robot description, xacro)
@@ -1,11 +1,4 @@
 <?xml version="1.0"?>
-<robot xmlns:xacro="http://www.ros.org/wiki/xacro" >
-    <!-- Trunk joint to base -->
-    <joint name="trunk_joint" type="fixed">
-        <parent link="base_link"/>
-        <child link="trunk"/>
-        <!--Origin defines translation child frame relative to parent frame. Translation is performed in parent frame.-->
-        <origin xyz="0 0 1.0" rpy="0 0 0"/>  <!--testing-->
-    </joint>
+<robot xmlns:xacro="http://www.ros.org/wiki/xacro" name = "meldog_trunk">
     <xacro:property name="trunk_base_length" value="0.8" />
     <xacro:property name="trunk_base_width" value="0.2" />
@@ -14,5 +7,5 @@
     <xacro:property name="trunk_actuators_width" value="0.2" />
     <xacro:property name="trunk_actuators_height" value="0.1" />
-    <link name="trunk">
+    <link name="trunk_link">
         <inertial>
             <origin xyz="0.0 0.0 0.0" rpy="0.0 0.0 0.0"/>

Commit message: Lower leg links and joints added

File: src/meldog_description/description/meldog_core.urdf.xacro (robot description, xacro)
@@ -3,4 +3,5 @@
     <!-- PI -->
     <xacro:property name="PI" value="3.1415926535897"/>
+    <!-- LINKS: -->
     <!-- Base link spawns in x= 0.0 y = 0.0 z = 0.0 -->
     <link name="base_link"></link>
@@ -13,4 +14,11 @@
     <xacro:hip_link position="back_left"/>
     <xacro:hip_link position="back_right"/>
+    <!-- Lower leg links -->
+    <xacro:include filename="lower_leg/lower_leg.urdf.xacro"/>
+    <xacro:lower_leg_link position="front_left"/>
+    <xacro:lower_leg_link position="front_right"/>
+    <xacro:lower_leg_link position="back_left"/>
+    <xacro:lower_leg_link position="back_right"/>
+    <!-- JOINTS: -->
     <!-- Base to Trunk joint -->
     <joint name="base_trunk_joint" type="fixed">
@@ -52,3 +60,35 @@
         <limit lower="-1.0" upper="1" effort="10.0" velocity="100.0"/>
     </joint>
+    <!-- Hip front left to Lower leg front left -->
+    <joint name="hip_lower_leg_front_left" type="revolute">
+        <origin xyz="${hip_length/2} ${hip_width/2 + lower_leg_radius} 0.0" rpy="0.0 0.0 0.0"/>
+        <parent link="hip_front_left_link"/>
+        <child link="lower_leg_front_left_link"/>
+        <axis xyz="0.0 1.0 0.0"/>
+        <limit lower="-1.0" upper="1.0" effort="10.0" velocity="100.0"/>
+    </joint>
+    <!-- Hip front right to Lower leg front right -->
+    <joint name="hip_lower_leg_front_right" type="revolute">
+        <origin xyz="${hip_length/2} ${-(hip_width/2 + lower_leg_radius)} 0.0" rpy="0.0 0.0 0.0"/>
+        <parent link="hip_front_right_link"/>
+        <child link="lower_leg_front_right_link"/>
+        <axis xyz="0.0 1.0 0.0"/>
+        <limit lower="-1.0" upper="1.0" effort="10.0" velocity="100.0"/>
+    </joint>
+    <!-- Hip back left to Lower leg back left -->
+    <joint name="hip_lower_leg_back_left" type="revolute">
+        <origin xyz="${hip_length/2} ${-(hip_width/2 + lower_leg_radius)} 0.0" rpy="0.0 0.0 0.0"/>
+        <parent link="hip_back_left_link"/>
+        <child link="lower_leg_back_left_link"/>
+        <axis xyz="0.0 1.0 0.0"/>
+        <limit lower="-1.0" upper="1.0" effort="10.0" velocity="100.0"/>
+    </joint>
+    <!-- Hip back right to Lower leg back right -->
+    <joint name="hip_lower_leg_back_right" type="revolute">
+        <origin xyz="${hip_length/2} ${hip_width/2 + lower_leg_radius} 0.0" rpy="0.0 0.0 0.0"/>
+        <parent link="hip_back_right_link"/>
+        <child link="lower_leg_back_right_link"/>
+        <axis xyz="0.0 1.0 0.0"/>
+        <limit lower="-1.0" upper="1.0" effort="10.0" velocity="100.0"/>
+    </joint>
 </robot>

Commit message: Added shank links and joints, changed lower_leg to thigh

File: src/meldog_description/description/meldog_core.urdf.xacro (robot description, xacro)
@@ -14,13 +14,19 @@
     <xacro:hip_link position="back_left"/>
     <xacro:hip_link position="back_right"/>
-    <!-- Lower leg links -->
-    <xacro:include filename="lower_leg/lower_leg.urdf.xacro"/>
-    <xacro:lower_leg_link position="front_left"/>
-    <xacro:lower_leg_link position="front_right"/>
-    <xacro:lower_leg_link position="back_left"/>
-    <xacro:lower_leg_link position="back_right"/>
+    <!-- Thigh links -->
+    <xacro:include filename="thigh/thigh.urdf.xacro"/>
+    <xacro:thigh_link position="front_left"/>
+    <xacro:thigh_link position="front_right"/>
+    <xacro:thigh_link position="back_left"/>
+    <xacro:thigh_link position="back_right"/>
+    <!-- Shank links -->
+    <xacro:include filename="shank/shank.urdf.xacro"/>
+    <xacro:shank_link position="front_left"/>
+    <xacro:shank_link position="front_right"/>
+    <xacro:shank_link position="back_left"/>
+    <xacro:shank_link position="back_right"/>
     <!-- JOINTS: -->
     <!-- Base to Trunk joint -->
-    <joint name="base_trunk_joint" type="fixed">
+    <joint name="BT_joint" type="fixed">
         <parent link="base_link"/>
         <child link="trunk_link"/>
@@ -29,5 +35,5 @@
     </joint>
     <!-- Trunk to Hip front left joint -->
-    <joint name="trunk_hip_front_left_joint" type="revolute">
+    <joint name="FLH_joint" type="revolute">
         <origin xyz="${trunk_actuators_length/2} ${trunk_base_width/2 + trunk_actuators_width/2} 0.0" rpy="0.0 0.0 0.0"/>
         <parent link="trunk_link"/>
@@ -37,5 +43,5 @@
     </joint>
     <!-- Trunk to Hip front right joint -->
-    <joint name="trunk_hip_front_right_joint" type="revolute">
+    <joint name="FRH_joint" type="revolute">
         <origin xyz="${trunk_actuators_length/2} ${-(trunk_base_width/2 + trunk_actuators_width/2)} 0.0" rpy="0.0 0.0 0.0"/>
         <parent link="trunk_link"/>
@@ -45,5 +51,5 @@
     </joint>
     <!-- Trunk to Hip back left joint -->
-    <joint name="trunk_hip_back_left_joint" type="revolute">
+    <joint name="BLH_joint" type="revolute">
         <origin xyz="${-trunk_actuators_length/2} ${trunk_base_width/2 + trunk_actuators_width/2} 0.0" rpy="0.0 0.0 ${PI}"/>
         <parent link="trunk_link"/>
@@ -53,5 +59,5 @@
     </joint>
     <!-- Trunk to Hip back right joint -->
-    <joint name="trunk_hip_back_right_joint" type="revolute">
+    <joint name="BRH_joint" type="revolute">
         <origin xyz="${-trunk_actuators_length/2} ${-(trunk_base_width/2 + trunk_actuators_width/2)} 0.0" rpy="0.0 0.0 ${PI}"/>
         <parent link="trunk_link"/>
@@ -60,33 +66,65 @@
         <limit lower="-1.0" upper="1" effort="10.0" velocity="100.0"/>
     </joint>
-    <!-- Hip front left to Lower leg front left -->
-    <joint name="hip_lower_leg_front_left" type="revolute">
-        <origin xyz="${hip_length/2} ${hip_width/2 + lower_leg_radius} 0.0" rpy="0.0 0.0 0.0"/>
+    <!-- Hip front left to Thigh front left -->
+    <joint name="FLT_joint" type="revolute">
+        <origin xyz="${hip_length/2} ${hip_width/2 + thigh_radius} 0.0" rpy="0.0 0.0 0.0"/>
         <parent link="hip_front_left_link"/>
-        <child link="lower_leg_front_left_link"/>
+        <child link="thigh_front_left_link"/>
         <axis xyz="0.0 1.0 0.0"/>
         <limit lower="-1.0" upper="1.0" effort="10.0" velocity="100.0"/>
     </joint>
-    <!-- Hip front right to Lower leg front right -->
-    <joint name="hip_lower_leg_front_right" type="revolute">
-        <origin xyz="${hip_length/2} ${-(hip_width/2 + lower_leg_radius)} 0.0" rpy="0.0 0.0 0.0"/>
+    <!-- Hip front right to Thigh front right -->
+    <joint name="FRT_joint" type="revolute">
+        <origin xyz="${hip_length/2} ${-(hip_width/2 + thigh_radius)} 0.0" rpy="0.0 0.0 0.0"/>
         <parent link="hip_front_right_link"/>
-        <child link="lower_leg_front_right_link"/>
+        <child link="thigh_front_right_link"/>
         <axis xyz="0.0 1.0 0.0"/>
         <limit lower="-1.0" upper="1.0" effort="10.0" velocity="100.0"/>
     </joint>
-    <!-- Hip back left to Lower leg back left -->
-    <joint name="hip_lower_leg_back_left" type="revolute">
-        <origin xyz="${hip_length/2} ${-(hip_width/2 + lower_leg_radius)} 0.0" rpy="0.0 0.0 0.0"/>
+    <!-- Hip back left to Thigh back left -->
+    <joint name="BLT_joint" type="revolute">
+        <origin xyz="${hip_length/2} ${-(hip_width/2 + thigh_radius)} 0.0" rpy="0.0 0.0 0.0"/>
         <parent link="hip_back_left_link"/>
-        <child link="lower_leg_back_left_link"/>
+        <child link="thigh_back_left_link"/>
         <axis xyz="0.0 1.0 0.0"/>
         <limit lower="-1.0" upper="1.0" effort="10.0" velocity="100.0"/>
     </joint>
-    <!-- Hip back right to Lower leg back right -->
-    <joint name="hip_lower_leg_back_right" type="revolute">
-        <origin xyz="${hip_length/2} ${hip_width/2 + lower_leg_radius} 0.0" rpy="0.0 0.0 0.0"/>
+    <!-- Hip back right to Thigh back right -->
+    <joint name="BRT_joint" type="revolute">
+        <origin xyz="${hip_length/2} ${hip_width/2 + thigh_radius} 0.0" rpy="0.0 0.0 0.0"/>
         <parent link="hip_back_right_link"/>
-        <child link="lower_leg_back_right_link"/>
+        <child link="thigh_back_right_link"/>
+        <axis xyz="0.0 1.0 0.0"/>
+        <limit lower="-1.0" upper="1.0" effort="10.0" velocity="100.0"/>
+    </joint>
+    <!-- Thigh front left to Shank front left -->
+    <joint name="FLS_joint" type="revolute">
+        <origin xyz="0.0 0.0 -${thigh_length}" rpy="0.0 0.0 0.0"/>
+        <parent link="thigh_front_left_link"/>
+        <child link="shank_front_left_link"/>
+        <axis xyz="0.0 1.0 0.0"/>
+        <limit lower="-1.0" upper="1.0" effort="10.0" velocity="100.0"/>
+    </joint>
+    <!-- Thigh front right to Shank front right -->
+    <joint name="FRS_joint" type="revolute">
+        <origin xyz="0.0 0.0 -${thigh_length}" rpy="0.0 0.0 0.0"/>
+        <parent link="thigh_front_right_link"/>
+        <child link="shank_front_right_link"/>
+        <axis xyz="0.0 1.0 0.0"/>
+        <limit lower="-1.0" upper="1.0" effort="10.0" velocity="100.0"/>
+    </joint>
+    <!-- Thigh back left to Shank back left -->
+    <joint name="BLS_joint" type="revolute">
+        <origin xyz="0.0 0.0 -${thigh_length}" rpy="0.0 0.0 0.0"/>
+        <parent link="thigh_back_left_link"/>
+        <child link="shank_back_left_link"/>
+        <axis xyz="0.0 1.0 0.0"/>
+        <limit lower="-1.0" upper="1.0" effort="10.0" velocity="100.0"/>
+    </joint>
+    <!-- Thigh back right to Shank back right -->
+    <joint name="BRS_joint" type="revolute">
+        <origin xyz="0.0 0.0 -${thigh_length}" rpy="0.0 0.0 0.0"/>
+        <parent link="thigh_back_right_link"/>
+        <child link="shank_back_right_link"/>
         <axis xyz="0.0 1.0 0.0"/>
         <limit lower="-1.0" upper="1.0" effort="10.0" velocity="100.0"/>

File: src/meldog_description/description/thigh/thigh.urdf.xacro (robot description, xacro)
@@ -1,8 +1,8 @@
 <?xml version="1.0"?>
-<robot xmlns:xacro="http://www.ros.org/wiki/xacro" name = "meldog_lower_leg">
-    <xacro:property name="lower_leg_length" value="0.2"/>
-    <xacro:property name="lower_leg_radius" value="0.05"/>
-    <xacro:macro name="lower_leg_link" params="position">
-        <link name="lower_leg_${position}_link">
+<robot xmlns:xacro="http://www.ros.org/wiki/xacro" name = "meldog_thigh">
+    <xacro:property name="thigh_length" value="0.5"/>
+    <xacro:property name="thigh_radius" value="0.05"/>
+    <xacro:macro name="thigh_link" params="position">
+        <link name="thigh_${position}_link">
             <inertial>
                 <origin xyz="0.0 0.0 0.0" rpy="0.0 0.0 0.0"/>
@@ -11,9 +11,9 @@
             </inertial>
             <visual name="">
-                <origin xyz="0.0 0.0 ${-lower_leg_length/2}" rpy="0.0 0.0 0.0"/>
+                <origin xyz="0.0 0.0 ${-thigh_length/2}" rpy="0.0 0.0 0.0"/>
                 <geometry>
-                    <cylinder radius="${lower_leg_radius}" length="${lower_leg_length}"/>
+                    <cylinder radius="${thigh_radius}" length="${thigh_length}"/>
                 </geometry>
-                <material name="lower_leg_${position}_link">
+                <material name="thigh_${position}_link">
                     <color rgba="0.0 1.0 0.0 1.0"/>
                     <texture filename=""/>

Commit message: Changed shank joints and added feet links and joints

File: src/meldog_description/description/meldog_core.urdf.xacro (robot description, xacro)
@@ -26,4 +26,10 @@
     <xacro:shank_link position="back_left"/>
     <xacro:shank_link position="back_right"/>
+    <!-- Feet links -->
+    <xacro:include filename="feet/feet.urdf.xacro"/>
+    <xacro:feet_link position="front_left"/>
+    <xacro:feet_link position="front_right"/>
+    <xacro:feet_link position="back_left"/>
+    <xacro:feet_link position="back_right"/>
     <!-- JOINTS: -->
     <!-- Base to Trunk joint -->
@@ -47,5 +53,5 @@
         <parent link="trunk_link"/>
         <child link="hip_front_right_link"/>
-        <axis xyz="1.0 0.0 0.0"/>
+        <axis xyz="-1.0 0.0 0.0"/>
         <limit lower="-1.0" upper="1" effort="10.0" velocity="100.0"/>
     </joint>
@@ -55,5 +61,5 @@
         <parent link="trunk_link"/>
         <child link="hip_back_left_link"/>
-        <axis xyz="1.0 0.0 0.0"/>
+        <axis xyz="-1.0 0.0 0.0"/>
         <limit lower="-1.0" upper="1" effort="10.0" velocity="100.0"/>
     </joint>
@@ -71,5 +77,5 @@
         <parent link="hip_front_left_link"/>
         <child link="thigh_front_left_link"/>
-        <axis xyz="0.0 1.0 0.0"/>
+        <axis xyz="0.0 -1.0 0.0"/>
         <limit lower="-1.0" upper="1.0" effort="10.0" velocity="100.0"/>
     </joint>
@@ -79,5 +85,5 @@
         <parent link="hip_front_right_link"/>
         <child link="thigh_front_right_link"/>
-        <axis xyz="0.0 1.0 0.0"/>
+        <axis xyz="0.0 -1.0 0.0"/>
         <limit lower="-1.0" upper="1.0" effort="10.0" velocity="100.0"/>
     </joint>
@@ -103,5 +109,5 @@
         <parent link="thigh_front_left_link"/>
         <child link="shank_front_left_link"/>
-        <axis xyz="0.0 1.0 0.0"/>
+        <axis xyz="0.0 -1.0 0.0"/>
         <limit lower="-1.0" upper="1.0" effort="10.0" velocity="100.0"/>
     </joint>
@@ -111,5 +117,5 @@
         <parent link="thigh_front_right_link"/>
         <child link="shank_front_right_link"/>
-        <axis xyz="0.0 1.0 0.0"/>
+        <axis xyz="0.0 -1.0 0.0"/>
         <limit lower="-1.0" upper="1.0" effort="10.0" velocity="100.0"/>
     </joint>
@@ -130,3 +136,27 @@
         <limit lower="-1.0" upper="1.0" effort="10.0" velocity="100.0"/>
     </joint>
+    <!-- Shank front left to Feet front left -->
+    <joint name="FLF_joint" type="fixed">
+        <origin xyz="0.0 0.0 ${-shank_length}" rpy="0.0 0.0 0.0"/>
+        <parent link="shank_front_left_link"/>
+        <child link="feet_front_left_link"/>
+    </joint>
+    <!-- Shank front right to Feet right left -->
+    <joint name="RLF_joint" type="fixed">
+        <origin xyz="0.0 0.0 ${-shank_length}" rpy="0.0 0.0 0.0"/>
+        <parent link="shank_front_right_link"/>
+        <child link="feet_front_right_link"/>
+    </joint>
+    <!-- Shank back left to Feet back left -->
+    <joint name="BLF_joint" type="fixed">
+        <origin xyz="0.0 0.0 ${-shank_length}" rpy="0.0 0.0 0.0"/>
+        <parent link="shank_back_left_link"/>
+        <child link="feet_back_left_link"/>
+    </joint>
+    <!-- Shank back right to Feet back right-->
+    <joint name="BRF_joint" type="fixed">
+        <origin xyz="0.0 0.0 ${-shank_length}" rpy="0.0 0.0 0.0"/>
+        <parent link="shank_back_right_link"/>
+        <child link="feet_back_right_link"/>
+    </joint>
 </robot>

Commit message: Deleted feed link, added only frames

File: src/meldog_description/description/meldog_core.urdf.xacro (robot description, xacro)
@@ -26,10 +26,9 @@
     <xacro:shank_link position="back_left"/>
     <xacro:shank_link position="back_right"/>
-    <!-- Feet links -->
-    <xacro:include filename="feet/feet.urdf.xacro"/>
-    <xacro:feet_link position="front_left"/>
-    <xacro:feet_link position="front_right"/>
-    <xacro:feet_link position="back_left"/>
-    <xacro:feet_link position="back_right"/>
+    <!-- Feet links (frames in the end of shank) -->
+    <link name="feet_front_left_link"></link>
+    <link name="feet_front_right_link"></link>
+    <link name="feet_back_left_link"></link>
+    <link name="feet_back_right_link"></link>
     <!-- JOINTS: -->
     <!-- Base to Trunk joint -->

File: src/meldog_description/description/shank/shank.urdf.xacro (robot description, xacro)
@@ -3,4 +3,5 @@
     <xacro:property name="shank_length" value="0.5"/>
     <xacro:property name="shank_radius" value="0.05"/>
+    <xacro:property name="feet_radius"  value ="0.08"/>
     <xacro:macro name="shank_link" params="position">
         <link name="shank_${position}_link">
@@ -15,6 +16,16 @@
                     <cylinder radius="${shank_radius}" length="${shank_length}"/>
                 </geometry>
-                <material name="shank_${position}_link">
+                <material name="yellow">
                     <color rgba="1.0 1.0 0.0 1.0"/>
+                    <texture filename=""/>
+                </material>
+            </visual>
+            <visual name="">
+                <origin xyz="0.0 0.0 ${-shank_length}" rpy="0.0 0.0 0.0"/>
+                <geometry>
+                    <sphere radius="${feet_radius}"/>
+                </geometry>
+                <material name="purple">
+                    <color rgba="1.0 0.0 1.0 1.0"/>
                     <texture filename=""/>
                 </material>
