Commit message: created separate files for each link in front legs

File: src/meldog_description/description/joints/meldog_joints.urdf.xacro (robot description, xacro)
@@ -1,95 +1,7 @@
 <?xml version="1.0"?>
-<robot name="meldog_core" xmlns:xacro="http://www.ros.org/wiki/xacro">
-    <xacro:include filename="base_properties.urdf.xacro" />
-    <xacro:include filename="macros/macros.urdf.xacro" />
-    <xacro:include filename="trunk.urdf.xacro" />
-    <!-- Left front leg links -->
-        <!-- Left front hip link -->
-        <xacro:include filename="links/hip/LFH_link.urdf.xacro"/>
-        <!-- Left front upper limb link -->
-        <xacro:include filename="links/upper_limb/LFUL_link.urdf.xacro"/>
-        <!-- Left front lower limb link -->
-        <xacro:include filename="links/lower_limb/LFLL_link.urdf.xacro"/>
-        <!-- Left front foot link -->
-        <xacro:include filename="links/foot/LFF_link.urdf.xacro"/>
-    <!-- Right front leg links -->
-        <!-- Right front hip link -->
-        <xacro:include filename="links/hip/RFH_link.urdf.xacro"/>
-        <!-- Right front upper limb link -->
-        <xacro:include filename="links/upper_limb/RFUL_link.urdf.xacro"/>
-        <!-- Right front lower limb link -->
-        <xacro:include filename="links/lower_limb/RFLL_link.urdf.xacro"/>
-        <!-- Right front foot link -->
-        <xacro:include filename="links/foot/RFF_link.urdf.xacro"/>
-    <!-- Left rear leg links -->
-    <xacro:link_macro
-        name="lr_hip_link"
-        vis_name="rear_left_hip.stl"
-        coll_name="rear_left_hip.stl"
-        m="${hip_mass}"
-        cm_x="${hip_cm_x}"
-        cm_y="${hip_cm_y}"
-        cm_z="${hip_cm_z}"
-        ixx="${hip_ixx}" ixy="${hip_ixy}" ixz="${hip_ixz}"
-                         iyy="${hip_iyy}" iyz="${hip_iyz}"
-                                          izz="${hip_izz}"/>
-    <xacro:link_macro
-        name="lr_upper_limb_link"
-        vis_name="upper_limb_test.stl"
-        coll_name="upper_limb_collision.stl"
-        m="${upper_limb_mass}"
-        cm_x="${upper_limb_cm_x}"
-        cm_y="${upper_limb_cm_y}"
-        cm_z="${upper_limb_cm_z}"
-        ixx="${upper_limb_ixx}" ixy="${upper_limb_ixy}" ixz="${upper_limb_ixz}"
-                                iyy="${upper_limb_iyy}" iyz="${upper_limb_iyz}"
-                                                        izz="${upper_limb_izz}"/>
-    <xacro:link_macro
-        name="lr_lower_limb_link"
-        vis_name="${lower_limb_vis_stl_name}"
-        coll_name="${lower_limb_coll_stl_name}"
-        m="${lower_limb_mass}"
-        cm_x="${lower_limb_cm_x}"
-        cm_y="${lower_limb_cm_y}"
-        cm_z="${lower_limb_cm_z}"
-        ixx="${lower_limb_ixx}" ixy="${lower_limb_ixy}" ixz="${lower_limb_ixz}"
-                                iyy="${lower_limb_iyy}" iyz="${lower_limb_iyz}"
-                                                        izz="${lower_limb_izz}"/>
-    <link name="lr_foot_link" />
-    <!-- Right rear leg links -->
-    <xacro:link_macro
-        name="rr_hip_link"
-        vis_name="rear_right_hip.stl"
-        coll_name="rear_right_hip.stl"
-        m="${hip_mass}"
-        cm_x="${hip_cm_x}"
-        cm_y="${hip_cm_y}"
-        cm_z="${hip_cm_z}"
-        ixx="${hip_ixx}" ixy="${hip_ixy}" ixz="${hip_ixz}"
-                         iyy="${hip_iyy}" iyz="${hip_iyz}"
-                                          izz="${hip_izz}"/>
-    <xacro:link_macro
-        name="rr_upper_limb_link"
-        vis_name="r_upper_limb_vis.stl"
-        coll_name="r_upper_limb_vis.stl"
-        m="${upper_limb_mass}"
-        cm_x="${upper_limb_cm_x}"
-        cm_y="${upper_limb_cm_y}"
-        cm_z="${upper_limb_cm_z}"
-        ixx="${upper_limb_ixx}" ixy="${upper_limb_ixy}" ixz="${upper_limb_ixz}"
-                                iyy="${upper_limb_iyy}" iyz="${upper_limb_iyz}"
-                                                        izz="${upper_limb_izz}"/>
-    <xacro:link_macro
-        name="rr_lower_limb_link"
-        vis_name="${lower_limb_vis_stl_name}"
-        coll_name="${lower_limb_coll_stl_name}"
-        m="${lower_limb_mass}"
-        cm_x="${lower_limb_cm_x}"
-        cm_y="${lower_limb_cm_y}"
-        cm_z="${lower_limb_cm_z}"
-        ixx="${lower_limb_ixx}" ixy="${lower_limb_ixy}" ixz="${lower_limb_ixz}"
-                                iyy="${lower_limb_iyy}" iyz="${lower_limb_iyz}"
-                                                        izz="${lower_limb_izz}"/>
-    <link name="rr_foot_link" />
+<robot xmlns:xacro="http://www.ros.org/wiki/xacro">
+    <xacro:include filename="../base_properties.urdf.xacro" />
+    <xacro:include filename="../links/meldog_links.urdf.xacro" />
+    <!-- <xacro:include filename="../trunk.urdf.xacro" /> -->
     <!-- left front leg joints -->
     <joint name="lf_hip_upper_limb_joint" type="revolute">

File: src/meldog_description/description/trunk.urdf.xacro (robot description, xacro)
@@ -1,4 +1,4 @@
 <?xml version="1.0"?>
-<robot xmlns:xacro="http://www.ros.org/wiki/xacro" name = "meldog_trunk">
+<robot xmlns:xacro="http://www.ros.org/wiki/xacro">
     <!-- Meldog trunk (3 simple boxes) -->
     <xacro:property name="trunk_base_length" value="0.8" />
