Commit message: added separate files for each link in rear legs

File: src/meldog_description/description/links/foot/LRF_link.urdf.xacro (robot description, xacro)
@@ -3,4 +3,4 @@
     <xacro:include filename="../../base_properties.urdf.xacro" />
     <xacro:include filename="../../macros/macros.urdf.xacro"/>
-    <link name="lr_foot_link" />
+    <link name="lf_foot_link" />
 </robot>

File: src/meldog_description/description/links/foot/RRF_link.urdf.xacro (robot description, xacro)
@@ -3,4 +3,4 @@
     <xacro:include filename="../../base_properties.urdf.xacro" />
     <xacro:include filename="../../macros/macros.urdf.xacro"/>
-    <link name="lr_foot_link" />
+    <link name="rr_foot_link" />
 </robot>

File: src/meldog_description/description/meldog_core.urdf.xacro (robot description, xacro)
@@ -3,5 +3,5 @@
     <xacro:include filename="base_properties.urdf.xacro" />
     <xacro:include filename="macros/macros.urdf.xacro" />
-    <xacro:include filename="trunk.urdf.xacro" />
+    <xacro:include filename="links/trunk.urdf.xacro" />
     <!-- Left front leg links -->
         <!-- Left front hip link -->
@@ -23,73 +23,21 @@
         <xacro:include filename="links/foot/RFF_link.urdf.xacro"/>
     <!-- Left rear leg links -->
-    <xacro:link_macro
-        name="lr_hip_link"
-        vis_name="rear_left_hip.stl"
-        coll_name="rear_left_hip.stl"
-        m="${hip_mass}"
-        cm_x="${hip_cm_x}"
-        cm_y="${hip_cm_y}"
-        cm_z="${hip_cm_z}"
-        ixx="${hip_ixx}" ixy="${hip_ixy}" ixz="${hip_ixz}"
-                         iyy="${hip_iyy}" iyz="${hip_iyz}"
-                                          izz="${hip_izz}"/>
-    <xacro:link_macro
-        name="lr_upper_limb_link"
-        vis_name="upper_limb_test.stl"
-        coll_name="upper_limb_collision.stl"
-        m="${upper_limb_mass}"
-        cm_x="${upper_limb_cm_x}"
-        cm_y="${upper_limb_cm_y}"
-        cm_z="${upper_limb_cm_z}"
-        ixx="${upper_limb_ixx}" ixy="${upper_limb_ixy}" ixz="${upper_limb_ixz}"
-                                iyy="${upper_limb_iyy}" iyz="${upper_limb_iyz}"
-                                                        izz="${upper_limb_izz}"/>
-    <xacro:link_macro
-        name="lr_lower_limb_link"
-        vis_name="${lower_limb_vis_stl_name}"
-        coll_name="${lower_limb_coll_stl_name}"
-        m="${lower_limb_mass}"
-        cm_x="${lower_limb_cm_x}"
-        cm_y="${lower_limb_cm_y}"
-        cm_z="${lower_limb_cm_z}"
-        ixx="${lower_limb_ixx}" ixy="${lower_limb_ixy}" ixz="${lower_limb_ixz}"
-                                iyy="${lower_limb_iyy}" iyz="${lower_limb_iyz}"
-                                                        izz="${lower_limb_izz}"/>
-    <link name="lr_foot_link" />
+        <!-- Left rear hip link -->
+        <xacro:include filename="links/hip/LRH_link.urdf.xacro"/>
+        <!-- Left rear upper limb link -->
+        <xacro:include filename="links/upper_limb/LRUL_link.urdf.xacro"/>
+        <!-- Left rear lower limb link -->
+        <xacro:include filename="links/lower_limb/LRLL_link.urdf.xacro"/>
+        <!-- Left rear foot link -->
+        <xacro:include filename="links/foot/LRF_link.urdf.xacro"/>
     <!-- Right rear leg links -->
-    <xacro:link_macro
-        name="rr_hip_link"
-        vis_name="rear_right_hip.stl"
-        coll_name="rear_right_hip.stl"
-        m="${hip_mass}"
-        cm_x="${hip_cm_x}"
-        cm_y="${hip_cm_y}"
-        cm_z="${hip_cm_z}"
-        ixx="${hip_ixx}" ixy="${hip_ixy}" ixz="${hip_ixz}"
-                         iyy="${hip_iyy}" iyz="${hip_iyz}"
-                                          izz="${hip_izz}"/>
-    <xacro:link_macro
-        name="rr_upper_limb_link"
-        vis_name="r_upper_limb_vis.stl"
-        coll_name="r_upper_limb_vis.stl"
-        m="${upper_limb_mass}"
-        cm_x="${upper_limb_cm_x}"
-        cm_y="${upper_limb_cm_y}"
-        cm_z="${upper_limb_cm_z}"
-        ixx="${upper_limb_ixx}" ixy="${upper_limb_ixy}" ixz="${upper_limb_ixz}"
-                                iyy="${upper_limb_iyy}" iyz="${upper_limb_iyz}"
-                                                        izz="${upper_limb_izz}"/>
-    <xacro:link_macro
-        name="rr_lower_limb_link"
-        vis_name="${lower_limb_vis_stl_name}"
-        coll_name="${lower_limb_coll_stl_name}"
-        m="${lower_limb_mass}"
-        cm_x="${lower_limb_cm_x}"
-        cm_y="${lower_limb_cm_y}"
-        cm_z="${lower_limb_cm_z}"
-        ixx="${lower_limb_ixx}" ixy="${lower_limb_ixy}" ixz="${lower_limb_ixz}"
-                                iyy="${lower_limb_iyy}" iyz="${lower_limb_iyz}"
-                                                        izz="${lower_limb_izz}"/>
-    <link name="rr_foot_link" />
+        <!-- Right rear hip link -->
+        <xacro:include filename="links/hip/RRH_link.urdf.xacro"/>
+        <!-- Right rear upper limb link -->
+        <xacro:include filename="links/upper_limb/RRUL_link.urdf.xacro"/>
+        <!-- Right rear lower limb link -->
+        <xacro:include filename="links/lower_limb/RRLL_link.urdf.xacro"/>
+        <!-- Right rear foot link -->
+        <xacro:include filename="links/foot/RRF_link.urdf.xacro"/>
     <!-- left front leg joints -->
     <joint name="lf_hip_upper_limb_joint" type="revolute">
