Commit message: added short link names

File: src/meldog_description/description/links/foot/LFF_link.urdf.xacro (robot description, xacro)
@@ -3,4 +3,4 @@
     <xacro:include filename="../../base_properties.urdf.xacro" />
     <xacro:include filename="../../macros/macros.urdf.xacro"/>
-    <link name="lr_foot_link" />
+    <link name="LFF_link" />
 </robot>

File: src/meldog_description/description/links/foot/LRF_link.urdf.xacro (robot description, xacro)
@@ -3,4 +3,4 @@
     <xacro:include filename="../../base_properties.urdf.xacro" />
     <xacro:include filename="../../macros/macros.urdf.xacro"/>
-    <link name="lf_foot_link" />
+    <link name="LRF_link" />
 </robot>

File: src/meldog_description/description/links/foot/RFF_link.urdf.xacro (robot description, xacro)
@@ -3,4 +3,4 @@
     <xacro:include filename="../../base_properties.urdf.xacro" />
     <xacro:include filename="../../macros/macros.urdf.xacro"/>
-    <link name="rf_foot_link" />
+    <link name="RFF_link" />
 </robot>

File: src/meldog_description/description/links/foot/RRF_link.urdf.xacro (robot description, xacro)
@@ -3,4 +3,4 @@
     <xacro:include filename="../../base_properties.urdf.xacro" />
     <xacro:include filename="../../macros/macros.urdf.xacro"/>
-    <link name="rr_foot_link" />
+    <link name="RRF_link" />
 </robot>

File: src/meldog_description/description/links/hip/LFH_link.urdf.xacro (robot description, xacro)
@@ -4,5 +4,5 @@
     <xacro:include filename="../../macros/macros.urdf.xacro"/>
     <xacro:link_macro
-        name="lf_hip_link"
+        name="LFH_link"
         vis_name="${hip_vis_stl_name}"
         coll_name="${hip_coll_stl_name}"

File: src/meldog_description/description/links/hip/LRH_link.urdf.xacro (robot description, xacro)
@@ -4,5 +4,5 @@
     <xacro:include filename="../../macros/macros.urdf.xacro"/>
     <xacro:link_macro
-        name="lr_hip_link"
+        name="LRH_link"
         vis_name="rear_left_hip.stl"
         coll_name="rear_left_hip_collision.stl"

File: src/meldog_description/description/links/hip/RFH_link.urdf.xacro (robot description, xacro)
@@ -4,5 +4,5 @@
     <xacro:include filename="../../macros/macros.urdf.xacro"/>
     <xacro:link_macro
-        name="rf_hip_link"
+        name="RFH_link"
         vis_name="front_right_hip.stl"
         coll_name="front_right_hip_collision.stl"

File: src/meldog_description/description/links/hip/RRH_link.urdf.xacro (robot description, xacro)
@@ -4,5 +4,5 @@
     <xacro:include filename="../../macros/macros.urdf.xacro"/>
     <xacro:link_macro
-        name="rr_hip_link"
+        name="RRH_link"
         vis_name="rear_right_hip.stl"
         coll_name="rear_right_hip_collision.stl"

File: src/meldog_description/description/links/lower_limb/LFLL_link.urdf.xacro (robot description, xacro)
@@ -4,5 +4,5 @@
     <xacro:include filename="../../macros/macros.urdf.xacro"/>
     <xacro:link_macro
-        name="lf_lower_limb_link"
+        name="LFLL_link"
         vis_name="${lower_limb_vis_stl_name}"
         coll_name="${lower_limb_coll_stl_name}"

File: src/meldog_description/description/links/lower_limb/LRLL_link.urdf.xacro (robot description, xacro)
@@ -4,5 +4,5 @@
     <xacro:include filename="../../macros/macros.urdf.xacro"/>
     <xacro:link_macro
-        name="lr_lower_limb_link"
+        name="LRLL_link"
         vis_name="${lower_limb_vis_stl_name}"
         coll_name="${lower_limb_coll_stl_name}"

File: src/meldog_description/description/links/lower_limb/RFLL_link.urdf.xacro (robot description, xacro)
@@ -4,5 +4,5 @@
     <xacro:include filename="../../macros/macros.urdf.xacro"/>
     <xacro:link_macro
-    name="rf_lower_limb_link"
+    name="RFLL_link"
     vis_name="${lower_limb_vis_stl_name}"
     coll_name="${lower_limb_coll_stl_name}"

File: src/meldog_description/description/links/lower_limb/RRLL_link.urdf.xacro (robot description, xacro)
@@ -4,5 +4,5 @@
     <xacro:include filename="../../macros/macros.urdf.xacro"/>
     <xacro:link_macro
-    name="rr_lower_limb_link"
+    name="RRLL_link"
     vis_name="${lower_limb_vis_stl_name}"
     coll_name="${lower_limb_coll_stl_name}"

File: src/meldog_description/description/links/upper_limb/LFUL_link.urdf.xacro (robot description, xacro)
@@ -4,5 +4,5 @@
     <xacro:include filename="../../macros/macros.urdf.xacro"/>
     <xacro:link_macro
-        name="lf_upper_limb_link"
+        name="LFUL_link"
         vis_name="${upper_limb_vis_stl_name}"
         coll_name="${upper_limb_coll_stl_name}"

File: src/meldog_description/description/links/upper_limb/LRUL_link.urdf.xacro (robot description, xacro)
@@ -4,5 +4,5 @@
     <xacro:include filename="../../macros/macros.urdf.xacro"/>
     <xacro:link_macro
-        name="lr_upper_limb_link"
+        name="LRUL_link"
         vis_name="upper_limb_test.stl"
         coll_name="upper_limb_collision.stl"

File: src/meldog_description/description/links/upper_limb/RFUL_link.urdf.xacro (robot description, xacro)
@@ -4,5 +4,5 @@
     <xacro:include filename="../../macros/macros.urdf.xacro"/>
     <xacro:link_macro
-        name="rf_upper_limb_link"
+        name="RFUL_link"
         vis_name="r_upper_limb_vis.stl"
         coll_name="upper_limb_collision.stl"

File: src/meldog_description/description/links/upper_limb/RRUL_link.urdf.xacro (robot description, xacro)
@@ -4,5 +4,5 @@
     <xacro:include filename="../../macros/macros.urdf.xacro"/>
     <xacro:link_macro
-        name="rr_upper_limb_link"
+        name="RRUL_link"
         vis_name="r_upper_limb_vis.stl"
         coll_name="upper_limb_collision.stl"

File: src/meldog_description/description/meldog_core.urdf.xacro (robot description, xacro)
@@ -42,6 +42,6 @@
     <!-- left front leg joints -->
     <joint name="lf_hip_upper_limb_joint" type="revolute">
-        <parent link="lf_hip_link" />
-        <child link="lf_upper_limb_link" />
+        <parent link="LFH_link" />
+        <child link="LFUL_link" />
         <origin xyz="${hip_upper_limb_x}
                      ${hip_upper_limb_y}
@@ -55,6 +55,6 @@
     </joint>
     <joint name="lf_upper_limb_lower_limb_joint" type="revolute">
-        <parent link="lf_upper_limb_link" />
-        <child link="lf_lower_limb_link" />
+        <parent link="LFUL_link" />
+        <child link="LFLL_link" />
         <origin xyz="0 0 ${-upper_limb_length}" rpy="0 0 0" />
         <limit lower="${upper_limb_lower_limb_lower_limit/180.0*pi}"
@@ -65,11 +65,11 @@
     </joint>
     <joint name="lf_lower_limb_foot_joint" type="fixed">
-        <parent link="lf_lower_limb_link" />
-        <child link="lf_foot_link" />
+        <parent link="LFLL_link" />
+        <child link="LFF_link" />
         <origin xyz="0 0 ${-lower_limb_length_to_foot}" rpy="0 0 0" />
     </joint>
     <joint name="lf_trunk_hip_joint" type="revolute">
         <parent link="trunk_link" />
-        <child link="lf_hip_link" />
+        <child link="LFH_link" />
         <origin xyz="${trunk_actuators_length/2.0} ${(trunk_base_width+trunk_actuators_width)/2.0} 0" rpy="0 0 0" />
         <limit lower="${trunk_hip_lower_limit/180.0*pi}"
@@ -82,5 +82,5 @@
     <joint name="rf_trunk_hip_joint" type="revolute">
         <parent link="trunk_link" />
-        <child link="rf_hip_link" />
+        <child link="RFH_link" />
         <origin xyz="${trunk_actuators_length/2.0} ${-(trunk_base_width+trunk_actuators_width)/2.0} 0" rpy="0 0 0" />
         <limit lower="${trunk_hip_lower_limit/180.0*pi}"
@@ -91,6 +91,6 @@
     </joint>
     <joint name="rf_hip_upper_limb_joint" type="revolute">
-        <parent link="rf_hip_link" />
-        <child link="rf_upper_limb_link" />
+        <parent link="RFH_link" />
+        <child link="RFUL_link" />
         <origin xyz="${hip_upper_limb_x}
                      ${-hip_upper_limb_y}
@@ -104,6 +104,6 @@
     </joint>
     <joint name="rf_upper_limb_lower_limb_joint" type="revolute">
-        <parent link="rf_upper_limb_link" />
-        <child link="rf_lower_limb_link" />
+        <parent link="RFUL_link" />
+        <child link="RFLL_link" />
         <origin xyz="0 0 ${-upper_limb_length}" rpy="0 0 0" />
         <limit lower="${upper_limb_lower_limb_lower_limit/180.0*pi}"
@@ -114,12 +114,12 @@
     </joint>
     <joint name="rf_lower_limb_foot_joint" type="fixed">
-        <parent link="rf_lower_limb_link" />
-        <child link="rf_foot_link" />
+        <parent link="RFLL_link" />
+        <child link="RFF_link" />
         <origin xyz="0 0 ${-lower_limb_length_to_foot}" rpy="0 0 0" />
     </joint>
     <!-- Left rear leg joints -->
     <joint name="lr_hip_upper_limb_joint" type="revolute">
-        <parent link="lr_hip_link" />
-        <child link="lr_upper_limb_link" />
+        <parent link="LRH_link" />
+        <child link="LRUL_link" />
         <origin xyz="${-hip_upper_limb_x}
                      ${hip_upper_limb_y}
@@ -133,6 +133,6 @@
     </joint>
     <joint name="lr_upper_limb_lower_limb_joint" type="revolute">
-        <parent link="lr_upper_limb_link" />
-        <child link="lr_lower_limb_link" />
+        <parent link="LRUL_link" />
+        <child link="LRLL_link" />
         <origin xyz="0 0 ${-upper_limb_length}" rpy="0 0 0" />
         <limit lower="${upper_limb_lower_limb_lower_limit/180.0*pi}"
@@ -143,11 +143,11 @@
     </joint>
     <joint name="lr_lower_limb_foot_joint" type="fixed">
-        <parent link="lr_lower_limb_link" />
-        <child link="lr_foot_link" />
+        <parent link="LRLL_link" />
+        <child link="LRF_link" />
         <origin xyz="0 0 ${-lower_limb_length_to_foot}" rpy="0 0 0" />
     </joint>
     <joint name="lr_trunk_hip_joint" type="revolute">
         <parent link="trunk_link" />
-        <child link="lr_hip_link" />
+        <child link="LRH_link" />
         <origin xyz="${-trunk_actuators_length/2.0} ${(trunk_base_width+trunk_actuators_width)/2.0} 0" rpy="0 0 0" />
         <limit lower="${trunk_hip_lower_limit/180.0*pi}"
@@ -160,5 +160,5 @@
     <joint name="rr_trunk_hip_joint" type="revolute">
         <parent link="trunk_link" />
-        <child link="rr_hip_link" />
+        <child link="RRH_link" />
         <origin xyz="${-trunk_actuators_length/2.0} ${-(trunk_base_width+trunk_actuators_width)/2.0} 0" rpy="0 0 0" />
         <limit lower="${trunk_hip_lower_limit/180.0*pi}"
@@ -169,6 +169,6 @@
     </joint>
     <joint name="rr_hip_upper_limb_joint" type="revolute">
-        <parent link="rr_hip_link" />
-        <child link="rr_upper_limb_link" />
+        <parent link="RRH_link" />
+        <child link="RRUL_link" />
         <origin xyz="${-hip_upper_limb_x}
                      ${-hip_upper_limb_y}
@@ -182,6 +182,6 @@
     </joint>
     <joint name="rr_upper_limb_lower_limb_joint" type="revolute">
-        <parent link="rr_upper_limb_link" />
-        <child link="rr_lower_limb_link" />
+        <parent link="RRUL_link" />
+        <child link="RRLL_link" />
         <origin xyz="0 0 ${-upper_limb_length}" rpy="0 0 0" />
         <limit lower="${upper_limb_lower_limb_lower_limit/180.0*pi}"
@@ -192,6 +192,6 @@
     </joint>
     <joint name="rr_lower_limb_foot_joint" type="fixed">
-        <parent link="rr_lower_limb_link" />
-        <child link="rr_foot_link" />
+        <parent link="RRLL_link" />
+        <child link="RRF_link" />
         <origin xyz="0 0 ${-lower_limb_length_to_foot}" rpy="0 0 0" />
     </joint>
