Commit message: Fixed trunk inertia

File: meldog_description/description/links/properties/T_properties.urdf.xacro (robot description, xacro)
@@ -19,9 +19,9 @@
         real robot trunk dimensions 72x34x14cm XYZ,
         here used inertia values fo cuboid 50x34x14 of uniform density to  better approximate real weight distribution-->
-        <xacro:property name="trunk_ixx" value="112667000.0"/> <!-- g*mm^2-->
+        <xacro:property name="trunk_ixx" value="112667.0"/> <!-- g*mm^2-->
         <xacro:property name="trunk_ixy" value="0"/> <!-- g*mm^2-->
         <xacro:property name="trunk_ixz" value="00"/> <!-- g*mm^2-->
-        <xacro:property name="trunk_iyy" value="224667000.0"/> <!-- g*mm^2-->
+        <xacro:property name="trunk_iyy" value="224667.0"/> <!-- g*mm^2-->
         <xacro:property name="trunk_iyz" value="0"/> <!-- g*mm^2-->
-        <xacro:property name="trunk_izz" value="304667000.0"/> <!-- g*mm^2-->
+        <xacro:property name="trunk_izz" value="304667.0"/> <!-- g*mm^2-->
 </robot>
