Commit message: Fixed contact broadcaster frame name

File: meldog_description/description/gazebo/gazebo_properties.urdf.xacro (robot description, xacro)
@@ -21,9 +21,9 @@
     <!-- Gazebo link parameters for feet -->
     <!-- Zoptymalizowane parametry kontaktu dla robota kroczącego -->
-    <xacro:property name="mu1_value_foot" value="0.8" /> <!-- Zwiększone tarcie, aby zapobiec mikro-uślizgom -->
-    <xacro:property name="mu2_value_foot" value="0.8" />
+    <xacro:property name="mu1_value_foot" value="1.8" /> <!-- Zwiększone tarcie, aby zapobiec mikro-uślizgom -->
+    <xacro:property name="mu2_value_foot" value="1.8" />
     <xacro:property name="kp_value_foot" value="1000000.0" /> <!-- Drastycznie zwiększona sztywność (10^6) -->
-    <xacro:property name="kd_value_foot" value="100.0" />     <!-- Zwiększone tłumienie, aby wygasić oscylacje -->
-    <xacro:property name="maxVel_value_foot" value="0.01" />   <!-- Ograniczenie maksymalnej prędkości naprawiania kontaktu -->
+    <xacro:property name="kd_value_foot" value="10.0" />     <!-- Zwiększone tłumienie, aby wygasić oscylacje -->
+    <xacro:property name="maxVel_value_foot" value="10.0" />   <!-- Ograniczenie maksymalnej prędkości naprawiania kontaktu -->
     <xacro:property name="minDepth_value_foot" value="0.001" /> <!-- Redukcja penetracji podłoża do zaledwie 1 milimetra -->
     <xacro:property name="dampingFactor_value_foot" value="0.01" />

File: meldog_description/description/gazebo/imu_gazebo_setup.urdf.xacro (robot description, xacro)
@@ -14,5 +14,5 @@
     <sensor name="imu_sensor" type="imu">
       <always_on>true</always_on>
-      <update_rate>1000</update_rate>  <!-- since controller manager runs on 1000Hz, the same goes with IMU-->
+      <update_rate>500</update_rate>  <!-- since controller manager runs on 1000Hz, the same goes with IMU-->
       <visualize>true</visualize>
       <imu>

Commit message: Fixed joint PD values

File: meldog_description/description/gazebo/gazebo_properties.urdf.xacro (robot description, xacro)
@@ -21,11 +21,15 @@
     <!-- Gazebo link parameters for feet -->
     <!-- Zoptymalizowane parametry kontaktu dla robota kroczącego -->
-    <xacro:property name="mu1_value_foot" value="1.8" /> <!-- Zwiększone tarcie, aby zapobiec mikro-uślizgom -->
-    <xacro:property name="mu2_value_foot" value="1.8" />
-    <xacro:property name="kp_value_foot" value="1000000.0" /> <!-- Drastycznie zwiększona sztywność (10^6) -->
-    <xacro:property name="kd_value_foot" value="10.0" />     <!-- Zwiększone tłumienie, aby wygasić oscylacje -->
-    <xacro:property name="maxVel_value_foot" value="10.0" />   <!-- Ograniczenie maksymalnej prędkości naprawiania kontaktu -->
-    <xacro:property name="minDepth_value_foot" value="0.001" /> <!-- Redukcja penetracji podłoża do zaledwie 1 milimetra -->
-    <xacro:property name="dampingFactor_value_foot" value="0.01" />
+    <!-- Higher friction coefficient to prevent shear micro-slips during trotting -->
+    <xacro:property name="mu1_value_foot" value="1.2" />
+    <xacro:property name="mu2_value_foot" value="1.2" />
+    <!-- Rigid floor contact stiffness (10^6) to eliminate soft sponge behavior -->
+    <xacro:property name="kp_value_foot" value="100000.0" />
+    <xacro:property name="kd_value_foot" value="10.0" />     <!-- Critical damping for 1e6 stiffness -->
+    <!-- Damp contact correction velocity to suppress acceleration shock spikes on IMU -->
+    <xacro:property name="maxVel_value_foot" value="0.01" />   <!-- 1 cm/s max correction speed -->
+    <!-- True 1 millimeter penetration depth limit -->
+    <xacro:property name="minDepth_value_foot" value="0.001" />
+    <xacro:property name="dampingFactor_value_foot" value="0.00" />
     <!-- <xacro:property name="mu1_value_foot" value="0.5" />
     <xacro:property name="mu2_value_foot" value="0.5" />

File: meldog_description/description/gazebo/imu_gazebo_setup.urdf.xacro (robot description, xacro)
@@ -14,5 +14,5 @@
     <sensor name="imu_sensor" type="imu">
       <always_on>true</always_on>
-      <update_rate>500</update_rate>  <!-- since controller manager runs on 1000Hz, the same goes with IMU-->
+      <update_rate>700</update_rate>  <!-- since controller manager runs on 1000Hz, the same goes with IMU-->
       <visualize>true</visualize>
       <imu>

File: meldog_description/description/joints/properties/H_joint_properties.urdf.xacro (robot description, xacro)
@@ -12,5 +12,5 @@
     <xacro:property name="H_velocity" value="${motor_max_vel*pi/30.0/actuator_reduction}" />
     <!-- Hip joint friction and damping -->
-    <xacro:property name="H_damping" value="0.05"/>
+    <xacro:property name="H_damping" value="0.08"/>
     <xacro:property name="H_friction" value="0.1312"/>
 </robot>

File: meldog_description/description/joints/properties/K_joint_properties.urdf.xacro (robot description, xacro)
@@ -10,5 +10,5 @@
     <xacro:property name="K_velocity" value="${motor_max_vel*pi/30.0/actuator_reduction}" />
     <!-- Knee joint friction and damping -->
-    <xacro:property name="K_damping" value="0.05"/>
+    <xacro:property name="K_damping" value="0.08"/>
     <xacro:property name="K_friction" value="0.1312"/>
 </robot>

File: meldog_description/description/joints/properties/T_joint_properties.urdf.xacro (robot description, xacro)
@@ -12,5 +12,5 @@
     <xacro:property name="T_velocity" value="${motor_max_vel*pi/30.0/actuator_reduction}" />
     <!-- Trunk joint friction and damping -->
-    <xacro:property name="T_damping" value="0.05"/>
+    <xacro:property name="T_damping" value="0.08"/>
     <xacro:property name="T_friction" value="0.1312"/>
 </robot>
